File: prius_gen2_kicad/connectors.sch (KiCad schematic (older format))
At the start: 10 parts

Commit message: schematics almost done
Parts:
- removed J?: Conn_02x10_Odd_Even, symbol Connector_Generic:Conn_02x10_Odd_Even
- removed J?: Conn_02x06_Odd_Even, symbol Connector_Generic:Conn_02x06_Odd_Even
- added J?: Conn_01x23, symbol Connector_Generic:Conn_01x23
- added J?: Conn_01x14, symbol Connector_Generic:Conn_01x14
Connections:
- net +12V: now also J?.20 (Pin_20)
- net +5V: now also R?.1, J?.19 (Pin_19), J?.6 (Pin_6); no longer R?.2
- net CAN_H: now also J?.18 (Pin_18)
- net CAN_L: now also J?.17 (Pin_17)
- net ENC_A: now also J?.3 (Pin_3)
- net ENC_B: now also J?.1 (Pin_1)
- net GIVA: now also J?.1 (Pin_1)
- net GIWA: now also J?.3 (Pin_3)
- net GND: now also R?.2, J?.12 (Pin_12), J?.2 (Pin_2), J?.21 (Pin_21); no longer R?.1
- net MFIV: now also J?.7 (Pin_7)
- net MIVA: now also J?.2 (Pin_2)
- net MIVT: now also J?.6 (Pin_6)
- net MIWA: now also J?.4 (Pin_4)
- net MTEMP+: now also J?.14 (Pin_14)
- net MTEMP-: now also J?.13 (Pin_13)
- net OUT_DCSW: now also J?.15 (Pin_15)
- net OUT_PRE: now also J?.16 (Pin_16)
- net R1: now also J?.4 (Pin_4)
- net R2: now also J?.5 (Pin_5)
- net SIG_BRAKE: now also J?.10 (Pin_10)
- net SIG_FWD: now also J?.11 (Pin_11)
- net SIG_REV: now also J?.12 (Pin_12)
- net SIG_START: now also J?.9 (Pin_9)
- net THROTTLE1: now also J?.7 (Pin_7)
- net THROTTLE2: now also J?.8 (Pin_8)
- net VH: now also J?.5 (Pin_5)
- net at U?.12 (O5): now also J?.9 (Pin_9)
- net at U?.13 (O4): now also J?.8 (Pin_8)
- net at U?.10 (O7): now also J?.11 (Pin_11)
- net at U?.11 (O6): now also J?.10 (Pin_10)
- net TIM1_BKIN: now reaches U?.16 (O1)
- no-connect marks 0 -> 8
Other:
- note added: "14pin\n776262-2\n1-776262-2\n\nMating plug:\n776273-2\n\n\n23pin\n\n776228-1\n\nMating plug:\n770680-1\n\n\nTerminals\n770854-1"
- moved on the sheet: C?, R?, U?

Commit message: fixed ERC
Parts:
- gave numbers to parts that had none: 10
Changed lines of the file:
@@
 P 3700 5350
 AR Path="/611D14C9" Ref="#PWR?"  Part="1"
-AR Path="/611C056E/611D14C9" Ref="#PWR?"  Part="1"
-F 0 "#PWR?" H 3700 5100 50  0001 C CNN
+AR Path="/611C056E/611D14C9" Ref="#PWR0131"  Part="1"
+F 0 "#PWR0131" H 3700 5100 50  0001 C CNN
 F 1 "GND" H 3705 5177 50  0000 C CNN
 F 2 "" H 3700 5350 50  0001 C CNN
@@
 P 3725 5225
 AR Path="/611D14DA" Ref="#PWR?"  Part="1"
-AR Path="/611C056E/611D14DA" Ref="#PWR?"  Part="1"
-F 0 "#PWR?" H 3725 5075 50  0001 C CNN
+AR Path="/611C056E/611D14DA" Ref="#PWR0132"  Part="1"
+F 0 "#PWR0132" H 3725 5075 50  0001 C CNN
 F 1 "+12V" V 3740 5353 50  0000 L CNN
 F 2 "" H 3725 5225 50  0001 C CNN
@@
 P 2800 2125
 AR Path="/611D14EF" Ref="R?"  Part="1"
-AR Path="/611C056E/611D14EF" Ref="R?"  Part="1"
-F 0 "R?" V 3007 2125 50  0000 C CNN
+AR Path="/611C056E/611D14EF" Ref="R22"  Part="1"
+F 0 "R22" V 3007 2125 50  0000 C CNN
 F 1 "510" V 2916 2125 50  0000 C CNN
 F 2 "" V 2730 2125 50  0001 C CNN
@@
 P 3200 3125
 AR Path="/611D14F6" Ref="#PWR?"  Part="1"
-AR Path="/611C056E/611D14F6" Ref="#PWR?"  Part="1"
-F 0 "#PWR?" H 3200 2875 50  0001 C CNN
+AR Path="/611C056E/611D14F6" Ref="#PWR0133"  Part="1"
+F 0 "#PWR0133" H 3200 2875 50  0001 C CNN
 F 1 "GND" H 3205 2952 50  0000 C CNN
 F 2 "" H 3200 3125 50  0001 C CNN
@@
 P 3550 2825
 AR Path="/611D14FC" Ref="R?"  Part="1"
-AR Path="/611C056E/611D14FC" Ref="R?"  Part="1"
-F 0 "R?" V 3343 2825 50  0000 C CNN
+AR Path="/611C056E/611D14FC" Ref="R23"  Part="1"
+F 0 "R23" V 3343 2825 50  0000 C CNN
 F 1 "220" V 3434 2825 50  0000 C CNN
 F 2 "" V 3480 2825 50  0001 C CNN
@@
 P 3200 2825
 AR Path="/611D1502" Ref="C?"  Part="1"
-AR Path="/611C056E/611D1502" Ref="C?"  Part="1"
-F 0 "C?" V 3452 2825 50  0000 C CNN
+AR Path="/611C056E/611D1502" Ref="C18"  Part="1"
+F 0 "C18" V 3452 2825 50  0000 C CNN
 F 1 "10uF" V 3361 2825 50  0000 C CNN
 F 2 "" H 3238 2675 50  0001 C CNN
@@
 P 2800 1850
 AR Path="/611D150B" Ref="#PWR?"  Part="1"
-AR Path="/611C056E/611D150B" Ref="#PWR?"  Part="1"
-F 0 "#PWR?" H 2800 1700 50  0001 C CNN
+AR Path="/611C056E/611D150B" Ref="#PWR0134"  Part="1"
+F 0 "#PWR0134" H 2800 1700 50  0001 C CNN
 F 1 "+5V" V 2815 1978 50  0000 L CNN
 F 2 "" H 2800 1850 50  0001 C CNN
@@
 P 3750 3825
 AR Path="/611D1521" Ref="#PWR?"  Part="1"
-AR Path="/611C056E/611D1521" Ref="#PWR?"  Part="1"
-F 0 "#PWR?" H 3750 3675 50  0001 C CNN
+AR Path="/611C056E/611D1521" Ref="#PWR0135"  Part="1"
+F 0 "#PWR0135" H 3750 3675 50  0001 C CNN
 F 1 "+5V" V 3765 3953 50  0000 L CNN
 F 2 "" H 3750 3825 50  0001 C CNN
@@
 MIVT
 $Comp
-L Transistor_Array:ULN2003A U?
+L Transistor_Array:ULN2003A U3
 U 1 1 6120D8B4
 P 7150 4125
-F 0 "U?" H 7150 4792 50  0000 C CNN
+F 0 "U3" H 7150 4792 50  0000 C CNN
 F 1 "ULN2003A" H 7150 4701 50  0000 C CNN
 F 2 "" H 7200 3575 50  0001 L CNN
@@
 	6600 3925 6750 3925
 $Comp
-L Device:R R?
+L Device:R R26
 U 1 1 6121673C
 P 6600 3100
-F 0 "R?" H 6670 3146 50  0000 L CNN
+F 0 "R26" H 6670 3146 50  0000 L CNN
 F 1 "10K" H 6670 3055 50  0000 L CNN
 F 2 "" V 6530 3100 50  0001 C CNN
@@
 $EndComp
 $Comp
-L power:+5V #PWR?
+L power:+5V #PWR0136
 U 1 1 61216AB4
 P 6600 2825
-F 0 "#PWR?" H 6600 2675 50  0001 C CNN
+F 0 "#PWR0136" H 6600 2675 50  0001 C CNN
 F 1 "+5V" H 6615 2998 50  0000 C CNN
 F 2 "" H 6600 2825 50  0001 C CNN
@@
 	6575 4525 6750 4525
 $Comp
-L power:GND #PWR?
+L power:GND #PWR0137
 U 1 1 6121F68A
 P 5825 4500
-F 0 "#PWR?" H 5825 4250 50  0001 C CNN
+F 0 "#PWR0137" H 5825 4250 50  0001 C CNN
 F 1 "GND" H 5830 4327 50  0000 C CNN
 F 2 "" H 5825 4500 50  0001 C CNN
@@
 $EndComp
 $Comp
-L Device:C C?
+L Device:C C19
 U 1 1 6121FA1F
 P 5525 4250
-F 0 "C?" H 5640 4296 50  0000 L CNN
+F 0 "C19" H 5640 4296 50  0000 L CNN
 F 1 "1nF" H 5640 4205 50  0000 L CNN
 F 2 "" H 5563 4100 50  0001 C CNN
@@
 $EndComp
 $Comp
-L Device:R R?
+L Device:R R25
 U 1 1 61220142
 P 5825 4250
-F 0 "R?" H 5895 4296 50  0000 L CNN
+F 0 "R25" H 5895 4296 50  0000 L CNN
 F 1 "4K7" H 5895 4205 50  0000 L CNN
 F 2 "" V 5755 4250 50  0001 C CNN
@@
 $EndComp
 $Comp
-L Device:R R?
+L Device:R R24
 U 1 1 612205C1
 P 5825 3800
-F 0 "R?" H 5895 3846 50  0000 L CNN
+F 0 "R24" H 5895 3846 50  0000 L CNN
 F 1 "10K" H 5895 3755 50  0000 L CNN
 F 2 "" V 5755 3800 50  0001 C CNN
@@
 	5825 4450 5825 4500
 $Comp
-L Connector_Generic:Conn_01x23 J?
+L Connector_Generic:Conn_01x23 J3
 U 1 1 60E8BF4D
 P 4175 4425
-F 0 "J?" H 4255 4467 50  0000 L CNN
+F 0 "J3" H 4255 4467 50  0000 L CNN
 F 1 "Conn_01x23" H 4255 4376 50  0000 L CNN
 F 2 "" H 4175 4425 50  0001 C CNN
@@
 $EndComp
 $Comp
-L Connector_Generic:Conn_01x14 J?
+L Connector_Generic:Conn_01x14 J4
 U 1 1 60E8DD9D
 P 8950 4125
-F 0 "J?" H 9030 4117 50  0000 L CNN
+F 0 "J4" H 9030 4117 50  0000 L CNN
 F 1 "Conn_01x14" H 9030 4026 50  0000 L CNN
 F 2 "" H 8950 4125 50  0001 C CNN
@@
 $EndComp
 $Comp
-L power:GND #PWR?
+L power:GND #PWR0138
 U 1 1 60EB22A1
 P 8600 4850
-F 0 "#PWR?" H 8600 4600 50  0001 C CNN
+F 0 "#PWR0138" H 8600 4600 50  0001 C CNN
 F 1 "GND" H 8605 4677 50  0000 C CNN
 F 2 "" H 8600 4850 50  0001 C CNN
@@
 P 3725 5125
 AR Path="/60F57711" Ref="#PWR?"  Part="1"
-AR Path="/611C056E/60F57711" Ref="#PWR?"  Part="1"
-F 0 "#PWR?" H 3725 4975 50  0001 C CNN
+AR Path="/611C056E/60F57711" Ref="#PWR0139"  Part="1"
+F 0 "#PWR0139" H 3725 4975 50  0001 C CNN
 F 1 "+5V" V 3740 5253 50  0000 L CNN
 F 2 "" H 3725 5125 50  0001 C CNN
@@
 	3975 5125 3725 5125
 Wire Wire Line
-	3725 5025 3975 5025
-Wire Wire Line
 	3725 4925 3975 4925
 Wire Wire Line
@@
 Text Notes 5275 6175 0    50   ~ 0
 14pin\n776262-2\n1-776262-2\n\nMating plug:\n776273-2\n\n\n23pin\n\n776228-1\n\nMating plug:\n770680-1\n\n\nTerminals\n770854-1
+Wire Wire Line
+	3975 5025 3725 5025
 $EndSCHEMATC

Commit message: started routing
Parts:
- C18, C19: footprint (none) -> Capacitor_SMD:C_0603_1608Metric
- J3: footprint (none) -> Downloads:TE_776228-1
- J4: footprint (none) -> Downloads:TE_776262-2
- R22, R23, R24, R25, R26: footprint (none) -> Resistor_SMD:R_0603_1608Metric
- U3: footprint (none) -> Package_SO:SOIC-16_4.55x10.3mm_P1.27mm
Changed lines of the file:
@@
 F 0 "R22" V 3007 2125 50  0000 C CNN
 F 1 "510" V 2916 2125 50  0000 C CNN
-F 2 "" V 2730 2125 50  0001 C CNN
+F 2 "Resistor_SMD:R_0603_1608Metric" V 2730 2125 50  0001 C CNN
 F 3 "~" H 2800 2125 50  0001 C CNN
 	1    2800 2125
@@
 F 0 "R23" V 3343 2825 50  0000 C CNN
 F 1 "220" V 3434 2825 50  0000 C CNN
-F 2 "" V 3480 2825 50  0001 C CNN
+F 2 "Resistor_SMD:R_0603_1608Metric" V 3480 2825 50  0001 C CNN
 F 3 "~" H 3550 2825 50  0001 C CNN
 	1    3550 2825
@@
 F 0 "C18" V 3452 2825 50  0000 C CNN
 F 1 "10uF" V 3361 2825 50  0000 C CNN
-F 2 "" H 3238 2675 50  0001 C CNN
+F 2 "Capacitor_SMD:C_0603_1608Metric" H 3238 2675 50  0001 C CNN
 F 3 "~" H 3200 2825 50  0001 C CNN
 	1    3200 2825
@@
 F 0 "U3" H 7150 4792 50  0000 C CNN
 F 1 "ULN2003A" H 7150 4701 50  0000 C CNN
-F 2 "" H 7200 3575 50  0001 L CNN
+F 2 "Package_SO:SOIC-16_4.55x10.3mm_P1.27mm" H 7200 3575 50  0001 L CNN
 F 3 "http://www.ti.com/lit/ds/symlink/uln2003a.pdf" H 7250 3925 50  0001 C CNN
 	1    7150 4125
@@
 F 0 "R26" H 6670 3146 50  0000 L CNN
 F 1 "10K" H 6670 3055 50  0000 L CNN
-F 2 "" V 6530 3100 50  0001 C CNN
+F 2 "Resistor_SMD:R_0603_1608Metric" V 6530 3100 50  0001 C CNN
 F 3 "~" H 6600 3100 50  0001 C CNN
 	1    6600 3100
@@
 F 0 "C19" H 5640 4296 50  0000 L CNN
 F 1 "1nF" H 5640 4205 50  0000 L CNN
-F 2 "" H 5563 4100 50  0001 C CNN
+F 2 "Capacitor_SMD:C_0603_1608Metric" H 5563 4100 50  0001 C CNN
 F 3 "~" H 5525 4250 50  0001 C CNN
 	1    5525 4250
@@
 F 0 "R25" H 5895 4296 50  0000 L CNN
 F 1 "4K7" H 5895 4205 50  0000 L CNN
-F 2 "" V 5755 4250 50  0001 C CNN
+F 2 "Resistor_SMD:R_0603_1608Metric" V 5755 4250 50  0001 C CNN
 F 3 "~" H 5825 4250 50  0001 C CNN
 	1    5825 4250
@@
 F 0 "R24" H 5895 3846 50  0000 L CNN
 F 1 "10K" H 5895 3755 50  0000 L CNN
-F 2 "" V 5755 3800 50  0001 C CNN
+F 2 "Resistor_SMD:R_0603_1608Metric" V 5755 3800 50  0001 C CNN
 F 3 "~" H 5825 3800 50  0001 C CNN
 	1    5825 3800
@@
 F 0 "J3" H 4255 4467 50  0000 L CNN
 F 1 "Conn_01x23" H 4255 4376 50  0000 L CNN
-F 2 "" H 4175 4425 50  0001 C CNN
+F 2 "Downloads:TE_776228-1" H 4175 4425 50  0001 C CNN
 F 3 "~" H 4175 4425 50  0001 C CNN
 	1    4175 4425
@@
 F 0 "J4" H 9030 4117 50  0000 L CNN
 F 1 "Conn_01x14" H 9030 4026 50  0000 L CNN
-F 2 "" H 8950 4125 50  0001 C CNN
+F 2 "Downloads:TE_776262-2" H 8950 4125 50  0001 C CNN
 F 3 "~" H 8950 4125 50  0001 C CNN
 	1    8950 4125
