File: prius_gen2_kicad/inputfilter.sch (KiCad schematic (older format))
At the start: 33 parts

Commit message: fixed ERC
Parts:
- gave numbers to parts that had none: 33

Commit message: started routing
Parts:
- C43, C44, C45, C46, C47, C48, C49, C51, C52: footprint (none) -> Capacitor_SMD:C_0603_1608Metric
- C50: value C -> 1u; footprint (none) -> Capacitor_SMD:C_0603_1608Metric
- JP2, JP3: footprint (none) -> Jumper:SolderJumper-2_P1.3mm_Open_TrianglePad1.0x1.5mm
- R41, R42, R43, R44, R45, R46, R47, R48, R49, R50, R51, R52, R53, R54, R55, R56, R57, R58, R59, R60, R61: footprint (none) -> Resistor_SMD:R_0603_1608Metric
Changed lines of the file:
@@
 F 0 "R46" V 3725 1750 50  0000 C CNN
 F 1 "3.3k" V 3725 1500 50  0000 C CNN
-F 2 "" V 3580 1650 50  0001 C CNN
+F 2 "Resistor_SMD:R_0603_1608Metric" V 3580 1650 50  0001 C CNN
 F 3 "~" H 3650 1650 50  0001 C CNN
 	1    3650 1650
@@
 F 0 "R47" V 3725 1975 50  0000 C CNN
 F 1 "3.3k" V 3725 1725 50  0000 C CNN
-F 2 "" V 3580 1875 50  0001 C CNN
+F 2 "Resistor_SMD:R_0603_1608Metric" V 3580 1875 50  0001 C CNN
 F 3 "~" H 3650 1875 50  0001 C CNN
 	1    3650 1875
@@
 F 0 "R48" V 3725 2200 50  0000 C CNN
 F 1 "3.3k" V 3725 1950 50  0000 C CNN
-F 2 "" V 3580 2100 50  0001 C CNN
+F 2 "Resistor_SMD:R_0603_1608Metric" V 3580 2100 50  0001 C CNN
 F 3 "~" H 3650 2100 50  0001 C CNN
 	1    3650 2100
@@
 F 0 "R49" V 3725 2425 50  0000 C CNN
 F 1 "3.3k" V 3725 2175 50  0000 C CNN
-F 2 "" V 3580 2325 50  0001 C CNN
+F 2 "Resistor_SMD:R_0603_1608Metric" V 3580 2325 50  0001 C CNN
 F 3 "~" H 3650 2325 50  0001 C CNN
 	1    3650 2325
@@
 F 0 "C45" H 4465 2796 50  0000 L CNN
 F 1 "1u" H 4465 2705 50  0000 L CNN
-F 2 "" H 4388 2600 50  0001 C CNN
+F 2 "Capacitor_SMD:C_0603_1608Metric" H 4388 2600 50  0001 C CNN
 F 3 "~" H 4350 2750 50  0001 C CNN
 	1    4350 2750
@@
 F 0 "R50" H 4720 2796 50  0000 L CNN
 F 1 "1.2k" H 4720 2705 50  0000 L CNN
-F 2 "" V 4580 2750 50  0001 C CNN
+F 2 "Resistor_SMD:R_0603_1608Metric" V 4580 2750 50  0001 C CNN
 F 3 "~" H 4650 2750 50  0001 C CNN
 	1    4650 2750
@@
 F 0 "C46" H 5090 2796 50  0000 L CNN
 F 1 "1u" H 5090 2705 50  0000 L CNN
-F 2 "" H 5013 2600 50  0001 C CNN
+F 2 "Capacitor_SMD:C_0603_1608Metric" H 5013 2600 50  0001 C CNN
 F 3 "~" H 4975 2750 50  0001 C CNN
 	1    4975 2750
@@
 F 0 "R51" H 5345 2796 50  0000 L CNN
 F 1 "1.2k" H 5345 2705 50  0000 L CNN
-F 2 "" V 5205 2750 50  0001 C CNN
+F 2 "Resistor_SMD:R_0603_1608Metric" V 5205 2750 50  0001 C CNN
 F 3 "~" H 5275 2750 50  0001 C CNN
 	1    5275 2750
@@
 F 0 "C47" H 5715 2796 50  0000 L CNN
 F 1 "1u" H 5715 2705 50  0000 L CNN
-F 2 "" H 5638 2600 50  0001 C CNN
+F 2 "Capacitor_SMD:C_0603_1608Metric" H 5638 2600 50  0001 C CNN
 F 3 "~" H 5600 2750 50  0001 C CNN
 	1    5600 2750
@@
 F 0 "R52" H 5970 2796 50  0000 L CNN
 F 1 "1.2k" H 5970 2705 50  0000 L CNN
-F 2 "" V 5830 2750 50  0001 C CNN
+F 2 "Resistor_SMD:R_0603_1608Metric" V 5830 2750 50  0001 C CNN
 F 3 "~" H 5900 2750 50  0001 C CNN
 	1    5900 2750
@@
 F 0 "C48" H 6340 2796 50  0000 L CNN
 F 1 "1u" H 6340 2705 50  0000 L CNN
-F 2 "" H 6263 2600 50  0001 C CNN
+F 2 "Capacitor_SMD:C_0603_1608Metric" H 6263 2600 50  0001 C CNN
 F 3 "~" H 6225 2750 50  0001 C CNN
 	1    6225 2750
@@
 F 0 "R53" H 6595 2796 50  0000 L CNN
 F 1 "1.2k" H 6595 2705 50  0000 L CNN
-F 2 "" V 6455 2750 50  0001 C CNN
+F 2 "Resistor_SMD:R_0603_1608Metric" V 6455 2750 50  0001 C CNN
 F 3 "~" H 6525 2750 50  0001 C CNN
 	1    6525 2750
@@
 F 0 "C49" H 6965 2796 50  0000 L CNN
 F 1 "1u" H 6965 2705 50  0000 L CNN
-F 2 "" H 6888 2600 50  0001 C CNN
+F 2 "Capacitor_SMD:C_0603_1608Metric" H 6888 2600 50  0001 C CNN
 F 3 "~" H 6850 2750 50  0001 C CNN
 	1    6850 2750
@@
 F 0 "R54" H 7220 2796 50  0000 L CNN
 F 1 "1.2k" H 7220 2705 50  0000 L CNN
-F 2 "" V 7080 2750 50  0001 C CNN
+F 2 "Resistor_SMD:R_0603_1608Metric" V 7080 2750 50  0001 C CNN
 F 3 "~" H 7150 2750 50  0001 C CNN
 	1    7150 2750
@@
 F 0 "R45" V 3725 1500 50  0000 C CNN
 F 1 "4.7k" V 3725 1250 50  0000 C CNN
-F 2 "" V 3580 1400 50  0001 C CNN
+F 2 "Resistor_SMD:R_0603_1608Metric" V 3580 1400 50  0001 C CNN
 F 3 "~" H 3650 1400 50  0001 C CNN
 	1    3650 1400
@@
 F 0 "R41" H 1545 4521 50  0000 L CNN
 F 1 "510" H 1545 4430 50  0000 L CNN
-F 2 "" V 1405 4475 50  0001 C CNN
+F 2 "Resistor_SMD:R_0603_1608Metric" V 1405 4475 50  0001 C CNN
 F 3 "~" H 1475 4475 50  0001 C CNN
 	1    1475 4475
@@
 F 0 "R43" V 1718 4700 50  0000 C CNN
 F 1 "10k" V 1809 4700 50  0000 C CNN
-F 2 "" V 1855 4700 50  0001 C CNN
+F 2 "Resistor_SMD:R_0603_1608Metric" V 1855 4700 50  0001 C CNN
 F 3 "~" H 1925 4700 50  0001 C CNN
 	1    1925 4700
@@
 F 0 "JP2" V 1429 4118 50  0000 L CNN
 F 1 "SolderJumper_2_Open" V 1520 4118 50  0000 L CNN
-F 2 "" H 1475 4050 50  0001 C CNN
+F 2 "Jumper:SolderJumper-2_P1.3mm_Open_TrianglePad1.0x1.5mm" H 1475 4050 50  0001 C CNN
 F 3 "~" H 1475 4050 50  0001 C CNN
 	1    1475 4050
@@
 F 0 "C43" H 2415 4946 50  0000 L CNN
 F 1 "1n" H 2415 4855 50  0000 L CNN
-F 2 "" H 2338 4750 50  0001 C CNN
+F 2 "Capacitor_SMD:C_0603_1608Metric" H 2338 4750 50  0001 C CNN
 F 3 "~" H 2300 4900 50  0001 C CNN
 	1    2300 4900
@@
 F 0 "R42" H 1545 5996 50  0000 L CNN
 F 1 "510" H 1545 5905 50  0000 L CNN
-F 2 "" V 1405 5950 50  0001 C CNN
+F 2 "Resistor_SMD:R_0603_1608Metric" V 1405 5950 50  0001 C CNN
 F 3 "~" H 1475 5950 50  0001 C CNN
 	1    1475 5950
@@
 F 0 "R44" V 1718 6175 50  0000 C CNN
 F 1 "10k" V 1809 6175 50  0000 C CNN
-F 2 "" V 1855 6175 50  0001 C CNN
+F 2 "Resistor_SMD:R_0603_1608Metric" V 1855 6175 50  0001 C CNN
 F 3 "~" H 1925 6175 50  0001 C CNN
 	1    1925 6175
@@
 F 0 "JP3" V 1429 5593 50  0000 L CNN
 F 1 "SolderJumper_2_Open" V 1520 5593 50  0000 L CNN
-F 2 "" H 1475 5525 50  0001 C CNN
+F 2 "Jumper:SolderJumper-2_P1.3mm_Open_TrianglePad1.0x1.5mm" H 1475 5525 50  0001 C CNN
 F 3 "~" H 1475 5525 50  0001 C CNN
 	1    1475 5525
@@
 F 0 "C44" H 2415 6421 50  0000 L CNN
 F 1 "1n" H 2415 6330 50  0000 L CNN
-F 2 "" H 2338 6225 50  0001 C CNN
+F 2 "Capacitor_SMD:C_0603_1608Metric" H 2338 6225 50  0001 C CNN
 F 3 "~" H 2300 6375 50  0001 C CNN
 	1    2300 6375
@@
 F 0 "R58" V 9882 3425 50  0000 C CNN
 F 1 "510" V 9791 3425 50  0000 C CNN
-F 2 "" V 9605 3425 50  0001 C CNN
+F 2 "Resistor_SMD:R_0603_1608Metric" V 9605 3425 50  0001 C CNN
 F 3 "~" H 9675 3425 50  0001 C CNN
 	1    9675 3425
@@
 F 0 "R59" V 9882 3750 50  0000 C CNN
 F 1 "510" V 9791 3750 50  0000 C CNN
-F 2 "" V 9605 3750 50  0001 C CNN
+F 2 "Resistor_SMD:R_0603_1608Metric" V 9605 3750 50  0001 C CNN
 F 3 "~" H 9675 3750 50  0001 C CNN
 	1    9675 3750
@@
 F 0 "R55" H 9520 4021 50  0000 L CNN
 F 1 "510" H 9520 3930 50  0000 L CNN
-F 2 "" V 9380 3975 50  0001 C CNN
+F 2 "Resistor_SMD:R_0603_1608Metric" V 9380 3975 50  0001 C CNN
 F 3 "~" H 9450 3975 50  0001 C CNN
 	1    9450 3975
@@
 P 9900 3975
 F 0 "C50" H 10015 4021 50  0000 L CNN
-F 1 "C" H 10015 3930 50  0000 L CNN
-F 2 "" H 9938 3825 50  0001 C CNN
+F 1 "1u" H 10015 3930 50  0000 L CNN
+F 2 "Capacitor_SMD:C_0603_1608Metric" H 9938 3825 50  0001 C CNN
 F 3 "~" H 9900 3975 50  0001 C CNN
 	1    9900 3975
@@
 F 0 "C52" H 10015 5721 50  0000 L CNN
 F 1 "1u" H 10015 5630 50  0000 L CNN
-F 2 "" H 9938 5525 50  0001 C CNN
+F 2 "Capacitor_SMD:C_0603_1608Metric" H 9938 5525 50  0001 C CNN
 F 3 "~" H 9900 5675 50  0001 C CNN
 	1    9900 5675
@@
 F 0 "R57" H 9520 5721 50  0000 L CNN
 F 1 "10k" H 9520 5630 50  0000 L CNN
-F 2 "" V 9380 5675 50  0001 C CNN
+F 2 "Resistor_SMD:R_0603_1608Metric" V 9380 5675 50  0001 C CNN
 F 3 "~" H 9450 5675 50  0001 C CNN
 	1    9450 5675
@@
 F 0 "R61" V 9882 5450 50  0000 C CNN
 F 1 "10k" V 9791 5450 50  0000 C CNN
-F 2 "" V 9605 5450 50  0001 C CNN
+F 2 "Resistor_SMD:R_0603_1608Metric" V 9605 5450 50  0001 C CNN
 F 3 "~" H 9675 5450 50  0001 C CNN
 	1    9675 5450
@@
 F 0 "C51" H 10015 4871 50  0000 L CNN
 F 1 "1u" H 10015 4780 50  0000 L CNN
-F 2 "" H 9938 4675 50  0001 C CNN
+F 2 "Capacitor_SMD:C_0603_1608Metric" H 9938 4675 50  0001 C CNN
 F 3 "~" H 9900 4825 50  0001 C CNN
 	1    9900 4825
@@
 F 0 "R56" H 9520 4871 50  0000 L CNN
 F 1 "10k" H 9520 4780 50  0000 L CNN
-F 2 "" V 9380 4825 50  0001 C CNN
+F 2 "Resistor_SMD:R_0603_1608Metric" V 9380 4825 50  0001 C CNN
 F 3 "~" H 9450 4825 50  0001 C CNN
 	1    9450 4825
@@
 F 0 "R60" V 9882 4600 50  0000 C CNN
 F 1 "10k" V 9791 4600 50  0000 C CNN
-F 2 "" V 9605 4600 50  0001 C CNN
+F 2 "Resistor_SMD:R_0603_1608Metric" V 9605 4600 50  0001 C CNN
 F 3 "~" H 9675 4600 50  0001 C CNN
 	1    9675 4600
