File: prius_gen2_kicad/level_shifting.sch (KiCad schematic (older format))
At the start: 23 parts

Commit message: schematics almost done
Parts:
- C? (x2): value 1nF -> 1n
- C? (x2): value 1uF -> 1u
Changed lines of the file:
@@
 $Descr A4 11693 8268
 encoding utf-8
-Sheet 2 5
+Sheet 2 7
 Title ""
 Date ""
@@
 AR Path="/611064E9/6111F5FD" Ref="C?"  Part="1"
 F 0 "C?" H 4540 2946 50  0000 L CNN
-F 1 "1nF" H 4540 2855 50  0000 L CNN
+F 1 "1n" H 4540 2855 50  0000 L CNN
 F 2 "" H 4463 2750 50  0001 C CNN
 F 3 "~" H 4425 2900 50  0001 C CNN
@@
 AR Path="/611064E9/6111F675" Ref="C?"  Part="1"
 F 0 "C?" H 4590 4221 50  0000 L CNN
-F 1 "1nF" H 4590 4130 50  0000 L CNN
+F 1 "1n" H 4590 4130 50  0000 L CNN
 F 2 "" H 4513 4025 50  0001 C CNN
 F 3 "~" H 4475 4175 50  0001 C CNN
@@
 AR Path="/611064E9/6111F69D" Ref="C?"  Part="1"
 F 0 "C?" H 4065 5246 50  0000 L CNN
-F 1 "1uF" H 4065 5155 50  0000 L CNN
+F 1 "1u" H 4065 5155 50  0000 L CNN
 F 2 "" H 3988 5050 50  0001 C CNN
 F 3 "~" H 3950 5200 50  0001 C CNN
@@
 AR Path="/611064E9/6111F6C4" Ref="C?"  Part="1"
 F 0 "C?" H 6215 5221 50  0000 L CNN
-F 1 "1uF" H 6215 5130 50  0000 L CNN
+F 1 "1u" H 6215 5130 50  0000 L CNN
 F 2 "" H 6138 5025 50  0001 C CNN
 F 3 "~" H 6100 5175 50  0001 C CNN

Commit message: fixed ERC
Parts:
- gave numbers to parts that had none: 21
Changed lines of the file:
@@
 P 5800 2550
 AR Path="/6111F5BF" Ref="U?"  Part="1"
-AR Path="/611064E9/6111F5BF" Ref="U?"  Part="1"
-F 0 "U?" H 5800 2917 50  0000 C CNN
+AR Path="/611064E9/6111F5BF" Ref="U2"  Part="1"
+F 0 "U2" H 5800 2917 50  0000 C CNN
 F 1 "MCP602" H 5800 2826 50  0000 C CNN
 F 2 "" H 5800 2550 50  0001 C CNN
@@
 P 5800 3825
 AR Path="/6111F5C5" Ref="U?"  Part="2"
-AR Path="/611064E9/6111F5C5" Ref="U?"  Part="2"
-F 0 "U?" H 5800 4192 50  0000 C CNN
+AR Path="/611064E9/6111F5C5" Ref="U2"  Part="2"
+F 0 "U2" H 5800 4192 50  0000 C CNN
 F 1 "MCP602" H 5800 4101 50  0000 C CNN
 F 2 "" H 5800 3825 50  0001 C CNN
@@
 P 7200 3575
 AR Path="/6111F5CB" Ref="U?"  Part="3"
-AR Path="/611064E9/6111F5CB" Ref="U?"  Part="3"
-F 0 "U?" H 7158 3621 50  0000 L CNN
+AR Path="/611064E9/6111F5CB" Ref="U2"  Part="3"
+F 0 "U2" H 7158 3621 50  0000 L CNN
 F 1 "MCP602" H 7158 3530 50  0000 L CNN
 F 2 "" H 7200 3575 50  0001 C CNN
@@
 P 7100 3200
 AR Path="/6111F5D1" Ref="#PWR?"  Part="1"
-AR Path="/611064E9/6111F5D1" Ref="#PWR?"  Part="1"
-F 0 "#PWR?" H 7100 3050 50  0001 C CNN
+AR Path="/611064E9/6111F5D1" Ref="#PWR0123"  Part="1"
+F 0 "#PWR0123" H 7100 3050 50  0001 C CNN
 F 1 "+5V" H 7115 3373 50  0000 C CNN
 F 2 "" H 7100 3200 50  0001 C CNN
@@
 P 7100 3975
 AR Path="/6111F5D7" Ref="#PWR?"  Part="1"
-AR Path="/611064E9/6111F5D7" Ref="#PWR?"  Part="1"
-F 0 "#PWR?" H 7100 3725 50  0001 C CNN
+AR Path="/611064E9/6111F5D7" Ref="#PWR0124"  Part="1"
+F 0 "#PWR0124" H 7100 3725 50  0001 C CNN
 F 1 "GND" H 7105 3802 50  0000 C CNN
 F 2 "" H 7100 3975 50  0001 C CNN
@@
 P 4775 2250
 AR Path="/6111F5E3" Ref="R?"  Part="1"
-AR Path="/611064E9/6111F5E3" Ref="R?"  Part="1"
-F 0 "R?" H 4845 2296 50  0000 L CNN
+AR Path="/611064E9/6111F5E3" Ref="R12"  Part="1"
+F 0 "R12" H 4845 2296 50  0000 L CNN
 F 1 "33K" H 4845 2205 50  0000 L CNN
 F 2 "" V 4705 2250 50  0001 C CNN
@@
 P 4125 2400
 AR Path="/6111F5EB" Ref="R?"  Part="1"
-AR Path="/611064E9/6111F5EB" Ref="R?"  Part="1"
-F 0 "R?" V 3918 2400 50  0000 C CNN
+AR Path="/611064E9/6111F5EB" Ref="R7"  Part="1"
+F 0 "R7" V 3918 2400 50  0000 C CNN
 F 1 "100K" V 4009 2400 50  0000 C CNN
 F 2 "" V 4055 2400 50  0001 C CNN
@@
 P 4125 2700
 AR Path="/6111F5F1" Ref="R?"  Part="1"
-AR Path="/611064E9/6111F5F1" Ref="R?"  Part="1"
-F 0 "R?" V 3918 2700 50  0000 C CNN
+AR Path="/611064E9/6111F5F1" Ref="R8"  Part="1"
+F 0 "R8" V 3918 2700 50  0000 C CNN
 F 1 "100K" V 4009 2700 50  0000 C CNN
 F 2 "" V 4055 2700 50  0001 C CNN
@@
 P 4425 2900
 AR Path="/6111F5FD" Ref="C?"  Part="1"
-AR Path="/611064E9/6111F5FD" Ref="C?"  Part="1"
-F 0 "C?" H 4540 2946 50  0000 L CNN
+AR Path="/611064E9/6111F5FD" Ref="C15"  Part="1"
+F 0 "C15" H 4540 2946 50  0000 L CNN
 F 1 "1n" H 4540 2855 50  0000 L CNN
 F 2 "" H 4463 2750 50  0001 C CNN
@@
 P 4425 3125
 AR Path="/6111F603" Ref="#PWR?"  Part="1"
-AR Path="/611064E9/6111F603" Ref="#PWR?"  Part="1"
-F 0 "#PWR?" H 4425 2875 50  0001 C CNN
+AR Path="/611064E9/6111F603" Ref="#PWR0125"  Part="1"
+F 0 "#PWR0125" H 4425 2875 50  0001 C CNN
 F 1 "GND" H 4430 2952 50  0000 C CNN
 F 2 "" H 4425 3125 50  0001 C CNN
@@
 P 4775 2675
 AR Path="/6111F60D" Ref="R?"  Part="1"
-AR Path="/611064E9/6111F60D" Ref="R?"  Part="1"
-F 0 "R?" H 4845 2721 50  0000 L CNN
+AR Path="/611064E9/6111F60D" Ref="R13"  Part="1"
+F 0 "R13" H 4845 2721 50  0000 L CNN
 F 1 "15K" H 4845 2630 50  0000 L CNN
 F 2 "" V 4705 2675 50  0001 C CNN
@@
 P 5225 2875
 AR Path="/6111F618" Ref="R?"  Part="1"
-AR Path="/611064E9/6111F618" Ref="R?"  Part="1"
-F 0 "R?" V 5018 2875 50  0000 C CNN
+AR Path="/611064E9/6111F618" Ref="R16"  Part="1"
+F 0 "R16" V 5018 2875 50  0000 C CNN
 F 1 "100K" V 5109 2875 50  0000 C CNN
 F 2 "" V 5155 2875 50  0001 C CNN
@@
 P 6150 2750
 AR Path="/6111F624" Ref="R?"  Part="1"
-AR Path="/611064E9/6111F624" Ref="R?"  Part="1"
-F 0 "R?" H 6080 2704 50  0000 R CNN
+AR Path="/611064E9/6111F624" Ref="R19"  Part="1"
+F 0 "R19" H 6080 2704 50  0000 R CNN
 F 1 "10K" H 6080 2795 50  0000 R CNN
 F 2 "" V 6080 2750 50  0001 C CNN
@@
 P 4775 2050
 AR Path="/6111F632" Ref="#PWR?"  Part="1"
-AR Path="/611064E9/6111F632" Ref="#PWR?"  Part="1"
-F 0 "#PWR?" H 4775 1900 50  0001 C CNN
+AR Path="/611064E9/6111F632" Ref="#PWR0126"  Part="1"
+F 0 "#PWR0126" H 4775 1900 50  0001 C CNN
 F 1 "+5V" H 4790 2223 50  0000 C CNN
 F 2 "" H 4775 2050 50  0001 C CNN
@@
 P 6150 4050
 AR Path="/6111F63D" Ref="R?"  Part="1"
-AR Path="/611064E9/6111F63D" Ref="R?"  Part="1"
-F 0 "R?" H 6080 4004 50  0000 R CNN
+AR Path="/611064E9/6111F63D" Ref="R20"  Part="1"
+F 0 "R20" H 6080 4004 50  0000 R CNN
 F 1 "10K" H 6080 4095 50  0000 R CNN
 F 2 "" V 6080 4050 50  0001 C CNN
@@
 P 5225 4150
 AR Path="/6111F643" Ref="R?"  Part="1"
-AR Path="/611064E9/6111F643" Ref="R?"  Part="1"
-F 0 "R?" V 5018 4150 50  0000 C CNN
+AR Path="/611064E9/6111F643" Ref="R17"  Part="1"
+F 0 "R17" V 5018 4150 50  0000 C CNN
 F 1 "100K" V 5109 4150 50  0000 C CNN
 F 2 "" V 5155 4150 50  0001 C CNN
@@
 P 4825 3925
 AR Path="/6111F649" Ref="R?"  Part="1"
-AR Path="/611064E9/6111F649" Ref="R?"  Part="1"
-F 0 "R?" H 4895 3971 50  0000 L CNN
+AR Path="/611064E9/6111F649" Ref="R15"  Part="1"
+F 0 "R15" H 4895 3971 50  0000 L CNN
 F 1 "15K" H 4895 3880 50  0000 L CNN
 F 2 "" V 4755 3925 50  0001 C CNN
@@
 P 4825 3525
 AR Path="/6111F64F" Ref="R?"  Part="1"
-AR Path="/611064E9/6111F64F" Ref="R?"  Part="1"
-F 0 "R?" H 4895 3571 50  0000 L CNN
+AR Path="/611064E9/6111F64F" Ref="R14"  Part="1"
+F 0 "R14" H 4895 3571 50  0000 L CNN
 F 1 "33K" H 4895 3480 50  0000 L CNN
 F 2 "" V 4755 3525 50  0001 C CNN
@@
 P 4175 3675
 AR Path="/6111F663" Ref="R?"  Part="1"
-AR Path="/611064E9/6111F663" Ref="R?"  Part="1"
-F 0 "R?" V 3968 3675 50  0000 C CNN
+AR Path="/611064E9/6111F663" Ref="R9"  Part="1"
+F 0 "R9" V 3968 3675 50  0000 C CNN
 F 1 "100K" V 4059 3675 50  0000 C CNN
 F 2 "" V 4105 3675 50  0001 C CNN
@@
 P 4175 3975
 AR Path="/6111F669" Ref="R?"  Part="1"
-AR Path="/611064E9/6111F669" Ref="R?"  Part="1"
-F 0 "R?" V 3968 3975 50  0000 C CNN
+AR Path="/611064E9/6111F669" Ref="R10"  Part="1"
+F 0 "R10" V 3968 3975 50  0000 C CNN
 F 1 "100K" V 4059 3975 50  0000 C CNN
 F 2 "" V 4105 3975 50  0001 C CNN
@@
 P 4475 4175
 AR Path="/6111F675" Ref="C?"  Part="1"
-AR Path="/611064E9/6111F675" Ref="C?"  Part="1"
-F 0 "C?" H 4590 4221 50  0000 L CNN
+AR Path="/611064E9/6111F675" Ref="C16"  Part="1"
+F 0 "C16" H 4590 4221 50  0000 L CNN
 F 1 "1n" H 4590 4130 50  0000 L CNN
 F 2 "" H 4513 4025 50  0001 C CNN
@@
 P 4475 4400
 AR Path="/6111F67D" Ref="#PWR?"  Part="1"
-AR Path="/611064E9/6111F67D" Ref="#PWR?"  Part="1"
-F 0 "#PWR?" H 4475 4150 50  0001 C CNN
+AR Path="/611064E9/6111F67D" Ref="#PWR0127"  Part="1"
+F 0 "#PWR0127" H 4475 4150 50  0001 C CNN
 F 1 "GND" H 4480 4227 50  0000 C CNN
 F 2 "" H 4475 4400 50  0001 C CNN
@@
 P 4825 3325
 AR Path="/6111F68C" Ref="#PWR?"  Part="1"
-AR Path="/611064E9/6111F68C" Ref="#PWR?"  Part="1"
-F 0 "#PWR?" H 4825 3175 50  0001 C CNN
+AR Path="/611064E9/6111F68C" Ref="#PWR0128"  Part="1"
+F 0 "#PWR0128" H 4825 3175 50  0001 C CNN
 F 1 "+5V" H 4840 3498 50  0000 C CNN
 F 2 "" H 4825 3325 50  0001 C CNN
@@
 P 3675 4950
 AR Path="/6111F697" Ref="R?"  Part="1"
-AR Path="/611064E9/6111F697" Ref="R?"  Part="1"
-F 0 "R?" V 3468 4950 50  0000 C CNN
+AR Path="/611064E9/6111F697" Ref="R6"  Part="1"
+F 0 "R6" V 3468 4950 50  0000 C CNN
 F 1 "10K" V 3559 4950 50  0000 C CNN
 F 2 "" V 3605 4950 50  0001 C CNN
@@
 P 3950 5200
 AR Path="/6111F69D" Ref="C?"  Part="1"
-AR Path="/611064E9/6111F69D" Ref="C?"  Part="1"
-F 0 "C?" H 4065 5246 50  0000 L CNN
+AR Path="/611064E9/6111F69D" Ref="C14"  Part="1"
+F 0 "C14" H 4065 5246 50  0000 L CNN
 F 1 "1u" H 4065 5155 50  0000 L CNN
 F 2 "" H 3988 5050 50  0001 C CNN
@@
 P 4300 5200
 AR Path="/6111F6A3" Ref="R?"  Part="1"
-AR Path="/611064E9/6111F6A3" Ref="R?"  Part="1"
-F 0 "R?" H 4370 5246 50  0000 L CNN
+AR Path="/611064E9/6111F6A3" Ref="R11"  Part="1"
+F 0 "R11" H 4370 5246 50  0000 L CNN
 F 1 "10K" H 4370 5155 50  0000 L CNN
 F 2 "" V 4230 5200 50  0001 C CNN
@@
 P 3950 5450
 AR Path="/6111F6A9" Ref="#PWR?"  Part="1"
-AR Path="/611064E9/6111F6A9" Ref="#PWR?"  Part="1"
-F 0 "#PWR?" H 3950 5200 50  0001 C CNN
+AR Path="/611064E9/6111F6A9" Ref="#PWR0129"  Part="1"
+F 0 "#PWR0129" H 3950 5200 50  0001 C CNN
 F 1 "GND" H 3955 5277 50  0000 C CNN
 F 2 "" H 3950 5450 50  0001 C CNN
@@
 P 5825 4925
 AR Path="/6111F6BE" Ref="R?"  Part="1"
-AR Path="/611064E9/6111F6BE" Ref="R?"  Part="1"
-F 0 "R?" V 5618 4925 50  0000 C CNN
+AR Path="/611064E9/6111F6BE" Ref="R18"  Part="1"
+F 0 "R18" V 5618 4925 50  0000 C CNN
 F 1 "10K" V 5709 4925 50  0000 C CNN
 F 2 "" V 5755 4925 50  0001 C CNN
@@
 P 6100 5175
 AR Path="/6111F6C4" Ref="C?"  Part="1"
-AR Path="/611064E9/6111F6C4" Ref="C?"  Part="1"
-F 0 "C?" H 6215 5221 50  0000 L CNN
+AR Path="/611064E9/6111F6C4" Ref="C17"  Part="1"
+F 0 "C17" H 6215 5221 50  0000 L CNN
 F 1 "1u" H 6215 5130 50  0000 L CNN
 F 2 "" H 6138 5025 50  0001 C CNN
@@
 P 6450 5175
 AR Path="/6111F6CA" Ref="R?"  Part="1"
-AR Path="/611064E9/6111F6CA" Ref="R?"  Part="1"
-F 0 "R?" H 6520 5221 50  0000 L CNN
+AR Path="/611064E9/6111F6CA" Ref="R21"  Part="1"
+F 0 "R21" H 6520 5221 50  0000 L CNN
 F 1 "10K" H 6520 5130 50  0000 L CNN
 F 2 "" V 6380 5175 50  0001 C CNN
@@
 P 6100 5425
 AR Path="/6111F6D0" Ref="#PWR?"  Part="1"
-AR Path="/611064E9/6111F6D0" Ref="#PWR?"  Part="1"
-F 0 "#PWR?" H 6100 5175 50  0001 C CNN
+AR Path="/611064E9/6111F6D0" Ref="#PWR0130"  Part="1"
+F 0 "#PWR0130" H 6100 5175 50  0001 C CNN
 F 1 "GND" H 6105 5252 50  0000 C CNN
 F 2 "" H 6100 5425 50  0001 C CNN

Commit message: started routing
Parts:
- C14, C15, C16, C17: footprint (none) -> Capacitor_SMD:C_0603_1608Metric
- R10, R11, R12, R13, R14, R15, R16, R17, R18, R19, R20, R21, R6, R7, R8, R9: footprint (none) -> Resistor_SMD:R_0603_1608Metric
- U2: footprint (none) -> Package_SO:SOIC-8-1EP_3.9x4.9mm_P1.27mm_EP2.29x3mm
Changed lines of the file:
@@
 F 0 "U2" H 5800 2917 50  0000 C CNN
 F 1 "MCP602" H 5800 2826 50  0000 C CNN
-F 2 "" H 5800 2550 50  0001 C CNN
+F 2 "Package_SO:SOIC-8-1EP_3.9x4.9mm_P1.27mm_EP2.29x3mm" H 5800 2550 50  0001 C CNN
 F 3 "http://ww1.microchip.com/downloads/en/DeviceDoc/21314g.pdf" H 5800 2550 50  0001 C CNN
 	1    5800 2550
@@
 F 0 "U2" H 5800 4192 50  0000 C CNN
 F 1 "MCP602" H 5800 4101 50  0000 C CNN
-F 2 "" H 5800 3825 50  0001 C CNN
+F 2 "Package_SO:SOIC-8-1EP_3.9x4.9mm_P1.27mm_EP2.29x3mm" H 5800 3825 50  0001 C CNN
 F 3 "http://ww1.microchip.com/downloads/en/DeviceDoc/21314g.pdf" H 5800 3825 50  0001 C CNN
 	2    5800 3825
@@
 F 0 "U2" H 7158 3621 50  0000 L CNN
 F 1 "MCP602" H 7158 3530 50  0000 L CNN
-F 2 "" H 7200 3575 50  0001 C CNN
+F 2 "Package_SO:SOIC-8-1EP_3.9x4.9mm_P1.27mm_EP2.29x3mm" H 7200 3575 50  0001 C CNN
 F 3 "http://ww1.microchip.com/downloads/en/DeviceDoc/21314g.pdf" H 7200 3575 50  0001 C CNN
 	3    7200 3575
@@
 F 0 "R12" H 4845 2296 50  0000 L CNN
 F 1 "33K" H 4845 2205 50  0000 L CNN
-F 2 "" V 4705 2250 50  0001 C CNN
+F 2 "Resistor_SMD:R_0603_1608Metric" V 4705 2250 50  0001 C CNN
 F 3 "~" H 4775 2250 50  0001 C CNN
 	1    4775 2250
@@
 F 0 "R7" V 3918 2400 50  0000 C CNN
 F 1 "100K" V 4009 2400 50  0000 C CNN
-F 2 "" V 4055 2400 50  0001 C CNN
+F 2 "Resistor_SMD:R_0603_1608Metric" V 4055 2400 50  0001 C CNN
 F 3 "~" H 4125 2400 50  0001 C CNN
 	1    4125 2400
@@
 F 0 "R8" V 3918 2700 50  0000 C CNN
 F 1 "100K" V 4009 2700 50  0000 C CNN
-F 2 "" V 4055 2700 50  0001 C CNN
+F 2 "Resistor_SMD:R_0603_1608Metric" V 4055 2700 50  0001 C CNN
 F 3 "~" H 4125 2700 50  0001 C CNN
 	1    4125 2700
@@
 F 0 "C15" H 4540 2946 50  0000 L CNN
 F 1 "1n" H 4540 2855 50  0000 L CNN
-F 2 "" H 4463 2750 50  0001 C CNN
+F 2 "Capacitor_SMD:C_0603_1608Metric" H 4463 2750 50  0001 C CNN
 F 3 "~" H 4425 2900 50  0001 C CNN
 	1    4425 2900
@@
 F 0 "R13" H 4845 2721 50  0000 L CNN
 F 1 "15K" H 4845 2630 50  0000 L CNN
-F 2 "" V 4705 2675 50  0001 C CNN
+F 2 "Resistor_SMD:R_0603_1608Metric" V 4705 2675 50  0001 C CNN
 F 3 "~" H 4775 2675 50  0001 C CNN
 	1    4775 2675
@@
 F 0 "R16" V 5018 2875 50  0000 C CNN
 F 1 "100K" V 5109 2875 50  0000 C CNN
-F 2 "" V 5155 2875 50  0001 C CNN
+F 2 "Resistor_SMD:R_0603_1608Metric" V 5155 2875 50  0001 C CNN
 F 3 "~" H 5225 2875 50  0001 C CNN
 	1    5225 2875
@@
 F 0 "R19" H 6080 2704 50  0000 R CNN
 F 1 "10K" H 6080 2795 50  0000 R CNN
-F 2 "" V 6080 2750 50  0001 C CNN
+F 2 "Resistor_SMD:R_0603_1608Metric" V 6080 2750 50  0001 C CNN
 F 3 "~" H 6150 2750 50  0001 C CNN
 	1    6150 2750
@@
 F 0 "R20" H 6080 4004 50  0000 R CNN
 F 1 "10K" H 6080 4095 50  0000 R CNN
-F 2 "" V 6080 4050 50  0001 C CNN
+F 2 "Resistor_SMD:R_0603_1608Metric" V 6080 4050 50  0001 C CNN
 F 3 "~" H 6150 4050 50  0001 C CNN
 	1    6150 4050
@@
 F 0 "R17" V 5018 4150 50  0000 C CNN
 F 1 "100K" V 5109 4150 50  0000 C CNN
-F 2 "" V 5155 4150 50  0001 C CNN
+F 2 "Resistor_SMD:R_0603_1608Metric" V 5155 4150 50  0001 C CNN
 F 3 "~" H 5225 4150 50  0001 C CNN
 	1    5225 4150
@@
 F 0 "R15" H 4895 3971 50  0000 L CNN
 F 1 "15K" H 4895 3880 50  0000 L CNN
-F 2 "" V 4755 3925 50  0001 C CNN
+F 2 "Resistor_SMD:R_0603_1608Metric" V 4755 3925 50  0001 C CNN
 F 3 "~" H 4825 3925 50  0001 C CNN
 	1    4825 3925
@@
 F 0 "R14" H 4895 3571 50  0000 L CNN
 F 1 "33K" H 4895 3480 50  0000 L CNN
-F 2 "" V 4755 3525 50  0001 C CNN
+F 2 "Resistor_SMD:R_0603_1608Metric" V 4755 3525 50  0001 C CNN
 F 3 "~" H 4825 3525 50  0001 C CNN
 	1    4825 3525
@@
 F 0 "R9" V 3968 3675 50  0000 C CNN
 F 1 "100K" V 4059 3675 50  0000 C CNN
-F 2 "" V 4105 3675 50  0001 C CNN
+F 2 "Resistor_SMD:R_0603_1608Metric" V 4105 3675 50  0001 C CNN
 F 3 "~" H 4175 3675 50  0001 C CNN
 	1    4175 3675
@@
 F 0 "R10" V 3968 3975 50  0000 C CNN
 F 1 "100K" V 4059 3975 50  0000 C CNN
-F 2 "" V 4105 3975 50  0001 C CNN
+F 2 "Resistor_SMD:R_0603_1608Metric" V 4105 3975 50  0001 C CNN
 F 3 "~" H 4175 3975 50  0001 C CNN
 	1    4175 3975
@@
 F 0 "C16" H 4590 4221 50  0000 L CNN
 F 1 "1n" H 4590 4130 50  0000 L CNN
-F 2 "" H 4513 4025 50  0001 C CNN
+F 2 "Capacitor_SMD:C_0603_1608Metric" H 4513 4025 50  0001 C CNN
 F 3 "~" H 4475 4175 50  0001 C CNN
 	1    4475 4175
@@
 F 0 "R6" V 3468 4950 50  0000 C CNN
 F 1 "10K" V 3559 4950 50  0000 C CNN
-F 2 "" V 3605 4950 50  0001 C CNN
+F 2 "Resistor_SMD:R_0603_1608Metric" V 3605 4950 50  0001 C CNN
 F 3 "~" H 3675 4950 50  0001 C CNN
 	1    3675 4950
@@
 F 0 "C14" H 4065 5246 50  0000 L CNN
 F 1 "1u" H 4065 5155 50  0000 L CNN
-F 2 "" H 3988 5050 50  0001 C CNN
+F 2 "Capacitor_SMD:C_0603_1608Metric" H 3988 5050 50  0001 C CNN
 F 3 "~" H 3950 5200 50  0001 C CNN
 	1    3950 5200
@@
 F 0 "R11" H 4370 5246 50  0000 L CNN
 F 1 "10K" H 4370 5155 50  0000 L CNN
-F 2 "" V 4230 5200 50  0001 C CNN
+F 2 "Resistor_SMD:R_0603_1608Metric" V 4230 5200 50  0001 C CNN
 F 3 "~" H 4300 5200 50  0001 C CNN
 	1    4300 5200
@@
 F 0 "R18" V 5618 4925 50  0000 C CNN
 F 1 "10K" V 5709 4925 50  0000 C CNN
-F 2 "" V 5755 4925 50  0001 C CNN
+F 2 "Resistor_SMD:R_0603_1608Metric" V 5755 4925 50  0001 C CNN
 F 3 "~" H 5825 4925 50  0001 C CNN
 	1    5825 4925
@@
 F 0 "C17" H 6215 5221 50  0000 L CNN
 F 1 "1u" H 6215 5130 50  0000 L CNN
-F 2 "" H 6138 5025 50  0001 C CNN
+F 2 "Capacitor_SMD:C_0603_1608Metric" H 6138 5025 50  0001 C CNN
 F 3 "~" H 6100 5175 50  0001 C CNN
 	1    6100 5175
@@
 F 0 "R21" H 6520 5221 50  0000 L CNN
 F 1 "10K" H 6520 5130 50  0000 L CNN
-F 2 "" V 6380 5175 50  0001 C CNN
+F 2 "Resistor_SMD:R_0603_1608Metric" V 6380 5175 50  0001 C CNN
 F 3 "~" H 6450 5175 50  0001 C CNN
 	1    6450 5175
