File: prius_gen2_kicad/resolver.sch (KiCad schematic (older format))
At the start: 10 parts

Commit message: schematics almost done
Parts:
- added C? (x2): 100n, symbol Device:C
- added C?: 22n, symbol Device:C
- added C?: 10u, symbol Device:C
- added R? (x2): 4.7k, symbol Device:R
- added U? (x2): TDA2822D, SOIC127P600X175-8N, symbol TDA2822D:TDA2822D
- R? (x3): value 3k3 -> 3.3k
Connections:
- net +5V: now also U?.2
- net GND: now also C?.1, C?.2, C?.2, U?.4, U?.6
- net at C?.1, R?.2: now also U?.7
- new net: C?.1, U?.8
- new net: C?.2, C?.2, U?.5
- new net: C?.1, R?.2 (x2)
- new net R1: R?.1, U?.1
- new net R2: R?.1, U?.3
Other:
- moved on the sheet: C?, R?

Commit message: fixed ERC
Parts:
- gave numbers to parts that had none: 17
Changed lines of the file:
@@
 TIM3_ETR
 $Comp
-L Device:R R?
+L Device:R R27
 U 1 1 60EAC28E
 P 4275 3050
-F 0 "R?" V 4068 3050 50  0000 C CNN
+F 0 "R27" V 4068 3050 50  0000 C CNN
 F 1 "3.3k" V 4159 3050 50  0000 C CNN
 F 2 "" V 4205 3050 50  0001 C CNN
@@
 $EndComp
 $Comp
-L Device:R R?
+L Device:R R28
 U 1 1 60EAC478
 P 4750 3050
-F 0 "R?" V 4543 3050 50  0000 C CNN
+F 0 "R28" V 4543 3050 50  0000 C CNN
 F 1 "3.3k" V 4634 3050 50  0000 C CNN
 F 2 "" V 4680 3050 50  0001 C CNN
@@
 $EndComp
 $Comp
-L Device:R R?
+L Device:R R29
 U 1 1 60EAC5BA
 P 5225 3050
-F 0 "R?" V 5018 3050 50  0000 C CNN
+F 0 "R29" V 5018 3050 50  0000 C CNN
 F 1 "3.3k" V 5109 3050 50  0000 C CNN
 F 2 "" V 5155 3050 50  0001 C CNN
@@
 $EndComp
 $Comp
-L Device:R R?
+L Device:R R30
 U 1 1 60EAC728
 P 5975 3275
-F 0 "R?" H 5905 3229 50  0000 R CNN
+F 0 "R30" H 5905 3229 50  0000 R CNN
 F 1 "10k" H 5905 3320 50  0000 R CNN
 F 2 "" V 5905 3275 50  0001 C CNN
@@
 	5075 3050 4975 3050
 $Comp
-L Device:C C?
+L Device:C C22
 U 1 1 60EACE0E
 P 4500 3300
-F 0 "C?" H 4615 3346 50  0000 L CNN
+F 0 "C22" H 4615 3346 50  0000 L CNN
 F 1 "22n" H 4615 3255 50  0000 L CNN
 F 2 "" H 4538 3150 50  0001 C CNN
@@
 $EndComp
 $Comp
-L Device:C C?
+L Device:C C23
 U 1 1 60EAD11D
 P 4975 3300
-F 0 "C?" H 5090 3346 50  0000 L CNN
+F 0 "C23" H 5090 3346 50  0000 L CNN
 F 1 "22n" H 5090 3255 50  0000 L CNN
 F 2 "" H 5013 3150 50  0001 C CNN
@@
 $EndComp
 $Comp
-L Device:C C?
+L Device:C C24
 U 1 1 60EAD325
 P 5450 3300
-F 0 "C?" H 5565 3346 50  0000 L CNN
+F 0 "C24" H 5565 3346 50  0000 L CNN
 F 1 "22n" H 5565 3255 50  0000 L CNN
 F 2 "" H 5488 3150 50  0001 C CNN
@@
 $EndComp
 $Comp
-L Device:C C?
+L Device:C C25
 U 1 1 60EADA96
 P 5650 3050
-F 0 "C?" V 5398 3050 50  0000 C CNN
+F 0 "C25" V 5398 3050 50  0000 C CNN
 F 1 "22n" V 5489 3050 50  0000 C CNN
 F 2 "" H 5688 2900 50  0001 C CNN
@@
 	5975 3050 5975 3125
 $Comp
-L power:GND #PWR?
+L power:GND #PWR0140
 U 1 1 60EAFA6D
 P 7025 3550
-F 0 "#PWR?" H 7025 3300 50  0001 C CNN
+F 0 "#PWR0140" H 7025 3300 50  0001 C CNN
 F 1 "GND" H 7030 3377 50  0000 C CNN
 F 2 "" H 7025 3550 50  0001 C CNN
@@
 Resolver Excitation
 $Comp
-L power:+5V #PWR?
+L power:+5V #PWR0141
 U 1 1 60EBE0BA
 P 4050 3900
-F 0 "#PWR?" H 4050 3750 50  0001 C CNN
+F 0 "#PWR0141" H 4050 3750 50  0001 C CNN
 F 1 "+5V" H 4065 4073 50  0000 C CNN
 F 2 "" H 4050 3900 50  0001 C CNN
@@
 $EndComp
 $Comp
-L Device:C C?
+L Device:C C20
 U 1 1 60EBE262
 P 3850 4150
-F 0 "C?" H 3965 4196 50  0000 L CNN
+F 0 "C20" H 3965 4196 50  0000 L CNN
 F 1 "1uF" H 3965 4105 50  0000 L CNN
 F 2 "" H 3888 4000 50  0001 C CNN
@@
 $EndComp
 $Comp
-L Device:C C?
+L Device:C C21
 U 1 1 60EBE45E
 P 4225 4150
-F 0 "C?" H 4340 4196 50  0000 L CNN
+F 0 "C21" H 4340 4196 50  0000 L CNN
 F 1 "100uF" H 4340 4105 50  0000 L CNN
 F 2 "" H 4263 4000 50  0001 C CNN
@@
 $EndComp
 $Comp
-L power:GND #PWR?
+L power:GND #PWR0142
 U 1 1 60EBEB3E
 P 4050 4400
-F 0 "#PWR?" H 4050 4150 50  0001 C CNN
+F 0 "#PWR0142" H 4050 4150 50  0001 C CNN
 F 1 "GND" H 4055 4227 50  0000 C CNN
 F 2 "" H 4050 4400 50  0001 C CNN
@@
 	3850 4300 3850 4350
 Wire Wire Line
-	3850 4350 4050 4350
-Wire Wire Line
-	4050 4350 4050 4400
-Wire Wire Line
-	4050 4350 4225 4350
-Wire Wire Line
 	4225 4350 4225 4300
-Connection ~ 4050 4350
 Wire Wire Line
 	4225 4000 4225 3950
@@
 Connection ~ 4050 3950
 $Comp
-L TDA2822D:TDA2822D U?
+L TDA2822D:TDA2822D U4
 U 1 1 61606D5B
 P 6925 2950
-F 0 "U?" H 7175 3100 50  0000 L CNN
+F 0 "U4" H 7175 3100 50  0000 L CNN
 F 1 "TDA2822D" H 7150 2825 50  0000 L CNN
 F 2 "SOIC127P600X175-8N" H 6925 2950 50  0001 L BNN
@@
 $EndComp
 $Comp
-L TDA2822D:TDA2822D U?
+L TDA2822D:TDA2822D U4
 U 2 1 616074FB
 P 6925 4250
-F 0 "U?" H 7200 4400 50  0000 C CNN
+F 0 "U4" H 7200 4400 50  0000 C CNN
 F 1 "TDA2822D" H 7275 4125 50  0000 C CNN
 F 2 "SOIC127P600X175-8N" H 6925 4250 50  0001 L BNN
@@
 	7800 2950 7575 2950
 $Comp
-L Device:R R?
+L Device:R R31
 U 1 1 6160E8C8
 P 7575 3175
-F 0 "R?" H 7645 3221 50  0000 L CNN
+F 0 "R31" H 7645 3221 50  0000 L CNN
 F 1 "4.7k" H 7645 3130 50  0000 L CNN
 F 2 "" V 7505 3175 50  0001 C CNN
@@
 $EndComp
 $Comp
-L Device:C C?
+L Device:C C28
 U 1 1 6160EF84
 P 7575 3575
-F 0 "C?" H 7690 3621 50  0000 L CNN
+F 0 "C28" H 7690 3621 50  0000 L CNN
 F 1 "100n" H 7690 3530 50  0000 L CNN
 F 2 "" H 7613 3425 50  0001 C CNN
@@
 $EndComp
 $Comp
-L power:GND #PWR?
+L power:GND #PWR0143
 U 1 1 61611699
 P 7575 3825
-F 0 "#PWR?" H 7575 3575 50  0001 C CNN
+F 0 "#PWR0143" H 7575 3575 50  0001 C CNN
 F 1 "GND" H 7580 3652 50  0000 C CNN
 F 2 "" H 7575 3825 50  0001 C CNN
@@
 	7575 3425 7575 3325
 $Comp
-L power:+5V #PWR?
+L power:+5V #PWR0144
 U 1 1 616132D9
 P 7025 2550
-F 0 "#PWR?" H 7025 2400 50  0001 C CNN
+F 0 "#PWR0144" H 7025 2400 50  0001 C CNN
 F 1 "+5V" H 7040 2723 50  0000 C CNN
 F 2 "" H 7025 2550 50  0001 C CNN
@@
 	7025 2550 7025 2650
 $Comp
-L Device:R R?
+L Device:R R32
 U 1 1 61615A70
 P 7575 4475
-F 0 "R?" H 7645 4521 50  0000 L CNN
+F 0 "R32" H 7645 4521 50  0000 L CNN
 F 1 "4.7k" H 7645 4430 50  0000 L CNN
 F 2 "" V 7505 4475 50  0001 C CNN
@@
 $EndComp
 $Comp
-L Device:C C?
+L Device:C C29
 U 1 1 61615B04
 P 7575 4875
-F 0 "C?" H 7690 4921 50  0000 L CNN
+F 0 "C29" H 7690 4921 50  0000 L CNN
 F 1 "100n" H 7690 4830 50  0000 L CNN
 F 2 "" H 7613 4725 50  0001 C CNN
@@
 $EndComp
 $Comp
-L power:GND #PWR?
+L power:GND #PWR0145
 U 1 1 61615B0E
 P 7575 5125
-F 0 "#PWR?" H 7575 4875 50  0001 C CNN
+F 0 "#PWR0145" H 7575 4875 50  0001 C CNN
 F 1 "GND" H 7580 4952 50  0000 C CNN
 F 2 "" H 7575 5125 50  0001 C CNN
@@
 Connection ~ 5975 3050
 $Comp
-L Device:C C?
+L Device:C C27
 U 1 1 6161DBD5
 P 6550 3825
-F 0 "C?" H 6665 3871 50  0000 L CNN
+F 0 "C27" H 6665 3871 50  0000 L CNN
 F 1 "22n" H 6665 3780 50  0000 L CNN
 F 2 "" H 6588 3675 50  0001 C CNN
@@
 $EndComp
 $Comp
-L Device:C C?
+L Device:C C26
 U 1 1 6161E12E
 P 6325 3825
-F 0 "C?" H 6200 3900 50  0000 L CNN
+F 0 "C26" H 6200 3900 50  0000 L CNN
 F 1 "10u" H 6350 3725 50  0000 L CNN
 F 2 "" H 6363 3675 50  0001 C CNN
@@
 Wire Notes Line
 	3400 5500 3400 2200
+Wire Wire Line
+	3850 4350 4050 4350
+Wire Wire Line
+	4050 4400 4050 4350
+Connection ~ 4050 4350
+Wire Wire Line
+	4050 4350 4225 4350
 $EndSCHEMATC

Commit message: started routing
Parts:
- C20, C22, C23, C24, C25, C26, C27, C28, C29: footprint (none) -> Capacitor_SMD:C_0603_1608Metric
- C21: footprint (none) -> Capacitor_SMD:C_Elec_6.3x7.7
- R27, R28, R29, R30, R31, R32: footprint (none) -> Resistor_SMD:R_0603_1608Metric
- U4: footprint SOIC127P600X175-8N -> Package_SO:SOIC-8-1EP_3.9x4.9mm_P1.27mm_EP2.29x3mm
Changed lines of the file:
@@
 F 0 "R27" V 4068 3050 50  0000 C CNN
 F 1 "3.3k" V 4159 3050 50  0000 C CNN
-F 2 "" V 4205 3050 50  0001 C CNN
+F 2 "Resistor_SMD:R_0603_1608Metric" V 4205 3050 50  0001 C CNN
 F 3 "~" H 4275 3050 50  0001 C CNN
 	1    4275 3050
@@
 F 0 "R28" V 4543 3050 50  0000 C CNN
 F 1 "3.3k" V 4634 3050 50  0000 C CNN
-F 2 "" V 4680 3050 50  0001 C CNN
+F 2 "Resistor_SMD:R_0603_1608Metric" V 4680 3050 50  0001 C CNN
 F 3 "~" H 4750 3050 50  0001 C CNN
 	1    4750 3050
@@
 F 0 "R29" V 5018 3050 50  0000 C CNN
 F 1 "3.3k" V 5109 3050 50  0000 C CNN
-F 2 "" V 5155 3050 50  0001 C CNN
+F 2 "Resistor_SMD:R_0603_1608Metric" V 5155 3050 50  0001 C CNN
 F 3 "~" H 5225 3050 50  0001 C CNN
 	1    5225 3050
@@
 F 0 "R30" H 5905 3229 50  0000 R CNN
 F 1 "10k" H 5905 3320 50  0000 R CNN
-F 2 "" V 5905 3275 50  0001 C CNN
+F 2 "Resistor_SMD:R_0603_1608Metric" V 5905 3275 50  0001 C CNN
 F 3 "~" H 5975 3275 50  0001 C CNN
 	1    5975 3275
@@
 F 0 "C22" H 4615 3346 50  0000 L CNN
 F 1 "22n" H 4615 3255 50  0000 L CNN
-F 2 "" H 4538 3150 50  0001 C CNN
+F 2 "Capacitor_SMD:C_0603_1608Metric" H 4538 3150 50  0001 C CNN
 F 3 "~" H 4500 3300 50  0001 C CNN
 	1    4500 3300
@@
 F 0 "C23" H 5090 3346 50  0000 L CNN
 F 1 "22n" H 5090 3255 50  0000 L CNN
-F 2 "" H 5013 3150 50  0001 C CNN
+F 2 "Capacitor_SMD:C_0603_1608Metric" H 5013 3150 50  0001 C CNN
 F 3 "~" H 4975 3300 50  0001 C CNN
 	1    4975 3300
@@
 F 0 "C24" H 5565 3346 50  0000 L CNN
 F 1 "22n" H 5565 3255 50  0000 L CNN
-F 2 "" H 5488 3150 50  0001 C CNN
+F 2 "Capacitor_SMD:C_0603_1608Metric" H 5488 3150 50  0001 C CNN
 F 3 "~" H 5450 3300 50  0001 C CNN
 	1    5450 3300
@@
 F 0 "C25" V 5398 3050 50  0000 C CNN
 F 1 "22n" V 5489 3050 50  0000 C CNN
-F 2 "" H 5688 2900 50  0001 C CNN
+F 2 "Capacitor_SMD:C_0603_1608Metric" H 5688 2900 50  0001 C CNN
 F 3 "~" H 5650 3050 50  0001 C CNN
 	1    5650 3050
@@
 F 0 "C20" H 3965 4196 50  0000 L CNN
 F 1 "1uF" H 3965 4105 50  0000 L CNN
-F 2 "" H 3888 4000 50  0001 C CNN
+F 2 "Capacitor_SMD:C_0603_1608Metric" H 3888 4000 50  0001 C CNN
 F 3 "~" H 3850 4150 50  0001 C CNN
 	1    3850 4150
@@
 F 0 "C21" H 4340 4196 50  0000 L CNN
 F 1 "100uF" H 4340 4105 50  0000 L CNN
-F 2 "" H 4263 4000 50  0001 C CNN
+F 2 "Capacitor_SMD:C_Elec_6.3x7.7" H 4263 4000 50  0001 C CNN
 F 3 "~" H 4225 4150 50  0001 C CNN
 	1    4225 4150
@@
 F 0 "U4" H 7175 3100 50  0000 L CNN
 F 1 "TDA2822D" H 7150 2825 50  0000 L CNN
-F 2 "SOIC127P600X175-8N" H 6925 2950 50  0001 L BNN
+F 2 "Package_SO:SOIC-8-1EP_3.9x4.9mm_P1.27mm_EP2.29x3mm" H 6925 2950 50  0001 L BNN
 F 3 "" H 6925 2950 50  0001 L BNN
 F 4 "IPC-7351B" H 6925 2950 50  0001 L BNN "STANDARD"
@@
 F 0 "U4" H 7200 4400 50  0000 C CNN
 F 1 "TDA2822D" H 7275 4125 50  0000 C CNN
-F 2 "SOIC127P600X175-8N" H 6925 4250 50  0001 L BNN
+F 2 "Package_SO:SOIC-8-1EP_3.9x4.9mm_P1.27mm_EP2.29x3mm" H 6925 4250 50  0001 L BNN
 F 3 "" H 6925 4250 50  0001 L BNN
 F 4 "IPC-7351B" H 6925 4250 50  0001 L BNN "STANDARD"
@@
 F 0 "R31" H 7645 3221 50  0000 L CNN
 F 1 "4.7k" H 7645 3130 50  0000 L CNN
-F 2 "" V 7505 3175 50  0001 C CNN
+F 2 "Resistor_SMD:R_0603_1608Metric" V 7505 3175 50  0001 C CNN
 F 3 "~" H 7575 3175 50  0001 C CNN
 	1    7575 3175
@@
 F 0 "C28" H 7690 3621 50  0000 L CNN
 F 1 "100n" H 7690 3530 50  0000 L CNN
-F 2 "" H 7613 3425 50  0001 C CNN
+F 2 "Capacitor_SMD:C_0603_1608Metric" H 7613 3425 50  0001 C CNN
 F 3 "~" H 7575 3575 50  0001 C CNN
 	1    7575 3575
@@
 F 0 "R32" H 7645 4521 50  0000 L CNN
 F 1 "4.7k" H 7645 4430 50  0000 L CNN
-F 2 "" V 7505 4475 50  0001 C CNN
+F 2 "Resistor_SMD:R_0603_1608Metric" V 7505 4475 50  0001 C CNN
 F 3 "~" H 7575 4475 50  0001 C CNN
 	1    7575 4475
@@
 F 0 "C29" H 7690 4921 50  0000 L CNN
 F 1 "100n" H 7690 4830 50  0000 L CNN
-F 2 "" H 7613 4725 50  0001 C CNN
+F 2 "Capacitor_SMD:C_0603_1608Metric" H 7613 4725 50  0001 C CNN
 F 3 "~" H 7575 4875 50  0001 C CNN
 	1    7575 4875
@@
 F 0 "C27" H 6665 3871 50  0000 L CNN
 F 1 "22n" H 6665 3780 50  0000 L CNN
-F 2 "" H 6588 3675 50  0001 C CNN
+F 2 "Capacitor_SMD:C_0603_1608Metric" H 6588 3675 50  0001 C CNN
 F 3 "~" H 6550 3825 50  0001 C CNN
 	1    6550 3825
@@
 F 0 "C26" H 6200 3900 50  0000 L CNN
 F 1 "10u" H 6350 3725 50  0000 L CNN
-F 2 "" H 6363 3675 50  0001 C CNN
+F 2 "Capacitor_SMD:C_0603_1608Metric" H 6363 3675 50  0001 C CNN
 F 3 "~" H 6325 3825 50  0001 C CNN
 	1    6325 3825
