File: prius_gen2_kicad/communication.sch (KiCad schematic (older format))
At the start: 6 parts

Commit message: schematics almost done
Parts:
- removed C?: 10uF, symbol Device:C
- removed C?: 1uF, symbol Device:C
- removed U?: SN65HVD230, Package_SO:SOIC-8_3.9x4.9mm_P1.27mm, symbol Interface_CAN_LIN:SN65HVD230
- added C? (x3): .1u, symbol Device:C
- added C?: 10u, symbol Device:C
- added D?: PESD1CAN-UX, symbol Device:D_TVS_x2_AAC
- added D?: LED, symbol Device:LED
- added J?: Conn_01x03_Male, symbol Connector:Conn_01x03_Male
- added R?: 10k, symbol Device:R
- added R?: 100, symbol Device:R
- added R?: R, symbol Device:R
- added SW?: RESET, symbol Switch:SW_Push
- added SW?: BOOT, symbol Switch:SW_Push
- added U?: TJA1051T-3, Package_SO:SOIC-8_3.9x4.9mm_P1.27mm, symbol Interface_CAN_LIN:TJA1051T-3
Connections:
- net labels added: +3.3V, +5V, CANH, CANL, ESP_RX, ESP_TX, RXDCAN, TXDCAN
- net labels removed: CANRX, CANTX, CAN_H, CAN_L, RX, TX
- wire segments 25 -> 67
- no-connect marks 0 -> 28
Other:
- note added: "CAN"
- note added: "ESP32 WiFi interface"
- note added: "Programming port"
- moved on the sheet: JP?, R?

Commit message: fixed ERC
Parts:
- gave numbers to parts that had none: 16
Changed lines of the file:
@@
 $EndDescr
 $Comp
-L Device:R R?
+L Device:R R33
 U 1 1 60EC4A3C
 P 2700 3450
-F 0 "R?" V 2493 3450 50  0000 C CNN
+F 0 "R33" V 2493 3450 50  0000 C CNN
 F 1 "120" V 2584 3450 50  0000 C CNN
 F 2 "" V 2630 3450 50  0001 C CNN
@@
 $EndComp
 $Comp
-L Jumper:SolderJumper_2_Open JP?
+L Jumper:SolderJumper_2_Open JP1
 U 1 1 60EC5424
 P 3250 3450
-F 0 "JP?" H 3250 3655 50  0000 C CNN
+F 0 "JP1" H 3250 3655 50  0000 C CNN
 F 1 "SolderJumper_2_Open" H 3250 3564 50  0000 C CNN
 F 2 "" H 3250 3450 50  0001 C CNN
@@
 	3100 3450 2850 3450
 $Comp
-L power:+3V3 #PWR?
+L power:+3V3 #PWR0146
 U 1 1 60EC75CC
 P 1975 4550
-F 0 "#PWR?" H 1975 4400 50  0001 C CNN
+F 0 "#PWR0146" H 1975 4400 50  0001 C CNN
 F 1 "+3V3" H 1990 4723 50  0000 C CNN
 F 2 "" H 1975 4550 50  0001 C CNN
@@
 $EndComp
 $Comp
-L RF_Module:ESP32-WROOM-32 U?
+L RF_Module:ESP32-WROOM-32 U6
 U 1 1 60EC899D
 P 7475 3825
-F 0 "U?" H 7025 2450 50  0000 C CNN
+F 0 "U6" H 7025 2450 50  0000 C CNN
 F 1 "ESP32-WROOM-32" H 7025 5200 50  0000 C CNN
 F 2 "RF_Module:ESP32-WROOM-32" H 7475 2325 50  0001 C CNN
@@
 $EndComp
 $Comp
-L power:GND #PWR?
+L power:GND #PWR0147
 U 1 1 60EC93A4
 P 7475 5325
-F 0 "#PWR?" H 7475 5075 50  0001 C CNN
+F 0 "#PWR0147" H 7475 5075 50  0001 C CNN
 F 1 "GND" H 7480 5152 50  0000 C CNN
 F 2 "" H 7475 5325 50  0001 C CNN
@@
 	7475 5325 7475 5225
 $Comp
-L power:+3V3 #PWR?
+L power:+3V3 #PWR0148
 U 1 1 60ECA1BD
 P 8250 1925
-F 0 "#PWR?" H 8250 1775 50  0001 C CNN
+F 0 "#PWR0148" H 8250 1775 50  0001 C CNN
 F 1 "+3V3" H 8265 2098 50  0000 C CNN
 F 2 "" H 8250 1925 50  0001 C CNN
@@
 	8075 2725 8325 2725
 $Comp
-L Interface_CAN_LIN:TJA1051T-3 U?
+L Interface_CAN_LIN:TJA1051T-3 U5
 U 1 1 60FE982B
 P 2675 4450
-F 0 "U?" H 2325 4075 50  0000 C CNN
+F 0 "U5" H 2325 4075 50  0000 C CNN
 F 1 "TJA1051T-3" H 2300 4800 50  0000 C CNN
 F 2 "Package_SO:SOIC-8_3.9x4.9mm_P1.27mm" H 2675 3950 50  0001 C CIN
@@
 $EndComp
 $Comp
-L power:+5V #PWR?
+L power:+5V #PWR0149
 U 1 1 60FEBEE7
 P 2675 3975
-F 0 "#PWR?" H 2675 3825 50  0001 C CNN
+F 0 "#PWR0149" H 2675 3825 50  0001 C CNN
 F 1 "+5V" H 2690 4148 50  0000 C CNN
 F 2 "" H 2675 3975 50  0001 C CNN
@@
 	1975 4550 2175 4550
 $Comp
-L power:GND #PWR?
+L power:GND #PWR0150
 U 1 1 60FF6A42
 P 2050 4750
-F 0 "#PWR?" H 2050 4500 50  0001 C CNN
+F 0 "#PWR0150" H 2050 4500 50  0001 C CNN
 F 1 "GND" H 2055 4577 50  0000 C CNN
 F 2 "" H 2050 4750 50  0001 C CNN
@@
 	2050 4650 2175 4650
 $Comp
-L power:GND #PWR?
+L power:GND #PWR0151
 U 1 1 60FF73C6
 P 2675 4975
-F 0 "#PWR?" H 2675 4725 50  0001 C CNN
+F 0 "#PWR0151" H 2675 4725 50  0001 C CNN
 F 1 "GND" H 2680 4802 50  0000 C CNN
 F 2 "" H 2675 4975 50  0001 C CNN
@@
 	2675 4975 2675 4850
 $Comp
-L Device:D_TVS_x2_AAC D?
+L Device:D_TVS_x2_AAC D2
 U 1 1 60FFAE8A
 P 3825 4425
-F 0 "D?" V 3871 4505 50  0000 L CNN
+F 0 "D2" V 3871 4505 50  0000 L CNN
 F 1 "PESD1CAN-UX" V 3780 4505 50  0000 L CNN
 F 2 "" H 3675 4425 50  0001 C CNN
@@
 	3825 4025 4200 4025
 $Comp
-L power:GND #PWR?
+L power:GND #PWR0152
 U 1 1 60FFFD04
 P 4100 4425
-F 0 "#PWR?" H 4100 4175 50  0001 C CNN
+F 0 "#PWR0152" H 4100 4175 50  0001 C CNN
 F 1 "GND" H 4105 4252 50  0000 C CNN
 F 2 "" H 4100 4425 50  0001 C CNN
@@
 ESP_RX
 $Comp
-L Switch:SW_Push SW?
+L Switch:SW_Push SW3
 U 1 1 6186DAB9
 P 6325 2850
-F 0 "SW?" V 6279 2998 50  0000 L CNN
+F 0 "SW3" V 6279 2998 50  0000 L CNN
 F 1 "RESET" V 6370 2998 50  0000 L CNN
 F 2 "" H 6325 3050 50  0001 C CNN
@@
 NoConn ~ 8075 4925
 $Comp
-L Device:C C?
+L Device:C C31
 U 1 1 6187C509
 P 7675 2125
-F 0 "C?" H 7790 2171 50  0000 L CNN
+F 0 "C31" H 7790 2171 50  0000 L CNN
 F 1 ".1u" H 7790 2080 50  0000 L CNN
 F 2 "" H 7713 1975 50  0001 C CNN
@@
 $EndComp
 $Comp
-L Device:C C?
+L Device:C C32
 U 1 1 6187C996
 P 8000 2125
-F 0 "C?" H 8115 2171 50  0000 L CNN
+F 0 "C32" H 8115 2171 50  0000 L CNN
 F 1 "10u" H 8115 2080 50  0000 L CNN
 F 2 "" H 8038 1975 50  0001 C CNN
@@
 $EndComp
 $Comp
-L power:GND #PWR?
+L power:GND #PWR0153
 U 1 1 6187CE43
 P 8200 2350
-F 0 "#PWR?" H 8200 2100 50  0001 C CNN
+F 0 "#PWR0153" H 8200 2100 50  0001 C CNN
 F 1 "GND" H 8205 2177 50  0000 C CNN
 F 2 "" H 8200 2350 50  0001 C CNN
@@
 Connection ~ 7675 1925
 $Comp
-L Device:R R?
+L Device:R R36
 U 1 1 618806A0
 P 8475 2100
-F 0 "R?" H 8545 2146 50  0000 L CNN
+F 0 "R36" H 8545 2146 50  0000 L CNN
 F 1 "10k" H 8545 2055 50  0000 L CNN
 F 2 "" V 8405 2100 50  0001 C CNN
@@
 	8075 2625 8475 2625
 $Comp
-L Device:C C?
+L Device:C C33
 U 1 1 61881D8E
 P 8775 2500
-F 0 "C?" H 8890 2546 50  0000 L CNN
+F 0 "C33" H 8890 2546 50  0000 L CNN
 F 1 ".1u" H 8890 2455 50  0000 L CNN
 F 2 "" H 8813 2350 50  0001 C CNN
@@
 $EndComp
 $Comp
-L power:GND #PWR?
+L power:GND #PWR0154
 U 1 1 61882C39
 P 8975 2750
-F 0 "#PWR?" H 8975 2500 50  0001 C CNN
+F 0 "#PWR0154" H 8975 2500 50  0001 C CNN
 F 1 "GND" H 8980 2577 50  0000 C CNN
 F 2 "" H 8975 2750 50  0001 C CNN
@@
 Connection ~ 8775 2250
 $Comp
-L Switch:SW_Push SW?
+L Switch:SW_Push SW4
 U 1 1 61882E01
 P 9200 2450
-F 0 "SW?" V 9154 2598 50  0000 L CNN
+F 0 "SW4" V 9154 2598 50  0000 L CNN
 F 1 "BOOT" V 9245 2598 50  0000 L CNN
 F 2 "" H 9200 2650 50  0001 C CNN
@@
 $EndComp
 $Comp
-L Device:LED D?
+L Device:LED D3
 U 1 1 6188DBD9
 P 8675 3325
-F 0 "D?" H 8668 3070 50  0000 C CNN
+F 0 "D3" H 8668 3070 50  0000 C CNN
 F 1 "LED" H 8668 3161 50  0000 C CNN
 F 2 "" H 8675 3325 50  0001 C CNN
@@
 $EndComp
 $Comp
-L Device:R R?
+L Device:R R35
 U 1 1 6188EDBA
 P 8350 3325
-F 0 "R?" V 8557 3325 50  0000 C CNN
+F 0 "R35" V 8557 3325 50  0000 C CNN
 F 1 "100" V 8466 3325 50  0000 C CNN
 F 2 "" V 8280 3325 50  0001 C CNN
@@
 $EndComp
 $Comp
-L power:GND #PWR?
+L power:GND #PWR0155
 U 1 1 6188F393
 P 9050 3400
-F 0 "#PWR?" H 9050 3150 50  0001 C CNN
+F 0 "#PWR0155" H 9050 3150 50  0001 C CNN
 F 1 "GND" H 9055 3227 50  0000 C CNN
 F 2 "" H 9050 3400 50  0001 C CNN
@@
 	8200 3325 8075 3325
 $Comp
-L Device:R R?
+L Device:R R34
 U 1 1 61891C81
 P 6475 2400
-F 0 "R?" H 6545 2446 50  0000 L CNN
+F 0 "R34" H 6545 2446 50  0000 L CNN
 F 1 "R" H 6545 2355 50  0000 L CNN
 F 2 "" V 6405 2400 50  0001 C CNN
@@
 $EndComp
 $Comp
-L power:+3.3V #PWR?
+L power:+3.3V #PWR0156
 U 1 1 618920DE
 P 6475 2175
-F 0 "#PWR?" H 6475 2025 50  0001 C CNN
+F 0 "#PWR0156" H 6475 2025 50  0001 C CNN
 F 1 "+3.3V" H 6490 2348 50  0000 C CNN
 F 2 "" H 6475 2175 50  0001 C CNN
@@
 $EndComp
 $Comp
-L Device:C C?
+L Device:C C30
 U 1 1 618924A7
 P 6075 2850
-F 0 "C?" H 5925 2925 50  0000 L CNN
+F 0 "C30" H 5925 2925 50  0000 L CNN
 F 1 ".1u" H 5925 2750 50  0000 L CNN
 F 2 "" H 6113 2700 50  0001 C CNN
@@
 $EndComp
 $Comp
-L power:GND #PWR?
+L power:GND #PWR0157
 U 1 1 618929D1
 P 6200 3200
-F 0 "#PWR?" H 6200 2950 50  0001 C CNN
+F 0 "#PWR0157" H 6200 2950 50  0001 C CNN
 F 1 "GND" H 6205 3027 50  0000 C CNN
 F 2 "" H 6200 3200 50  0001 C CNN
@@
 	6475 2625 6875 2625
 $Comp
-L Connector:Conn_01x03_Male J?
+L Connector:Conn_01x03_Male J5
 U 1 1 618C86EF
 P 8750 5025
-F 0 "J?" H 8858 5306 50  0000 C CNN
+F 0 "J5" H 8858 5306 50  0000 C CNN
 F 1 "Conn_01x03_Male" H 8858 5215 50  0000 C CNN
 F 2 "" H 8750 5025 50  0001 C CNN
@@
 $EndComp
 $Comp
-L power:GND #PWR?
+L power:GND #PWR0158
 U 1 1 618C8929
 P 9200 5275
-F 0 "#PWR?" H 9200 5025 50  0001 C CNN
+F 0 "#PWR0158" H 9200 5025 50  0001 C CNN
 F 1 "GND" H 9205 5102 50  0000 C CNN
 F 2 "" H 9200 5275 50  0001 C CNN

Commit message: started routing
Parts:
- C30, C31, C32, C33: footprint (none) -> Capacitor_SMD:C_0603_1608Metric
- D2: footprint (none) -> Package_TO_SOT_SMD:SOT-323_SC-70
- D3: footprint (none) -> LED_SMD:LED_0603_1608Metric_Castellated
- JP1: footprint (none) -> Jumper:SolderJumper-2_P1.3mm_Open_TrianglePad1.0x1.5mm
- R33, R34, R35, R36: footprint (none) -> Resistor_SMD:R_0603_1608Metric
- SW3, SW4: footprint (none) -> Button_Switch_SMD:SW_SPST_EVQQ2
Changed lines of the file:
@@
 F 0 "R33" V 2493 3450 50  0000 C CNN
 F 1 "120" V 2584 3450 50  0000 C CNN
-F 2 "" V 2630 3450 50  0001 C CNN
+F 2 "Resistor_SMD:R_0603_1608Metric" V 2630 3450 50  0001 C CNN
 F 3 "~" H 2700 3450 50  0001 C CNN
 	1    2700 3450
@@
 F 0 "JP1" H 3250 3655 50  0000 C CNN
 F 1 "SolderJumper_2_Open" H 3250 3564 50  0000 C CNN
-F 2 "" H 3250 3450 50  0001 C CNN
+F 2 "Jumper:SolderJumper-2_P1.3mm_Open_TrianglePad1.0x1.5mm" H 3250 3450 50  0001 C CNN
 F 3 "~" H 3250 3450 50  0001 C CNN
 	1    3250 3450
@@
 F 0 "D2" V 3871 4505 50  0000 L CNN
 F 1 "PESD1CAN-UX" V 3780 4505 50  0000 L CNN
-F 2 "" H 3675 4425 50  0001 C CNN
+F 2 "Package_TO_SOT_SMD:SOT-323_SC-70" H 3675 4425 50  0001 C CNN
 F 3 "~" H 3675 4425 50  0001 C CNN
 	1    3825 4425
@@
 F 0 "SW3" V 6279 2998 50  0000 L CNN
 F 1 "RESET" V 6370 2998 50  0000 L CNN
-F 2 "" H 6325 3050 50  0001 C CNN
+F 2 "Button_Switch_SMD:SW_SPST_EVQQ2" H 6325 3050 50  0001 C CNN
 F 3 "~" H 6325 3050 50  0001 C CNN
 	1    6325 2850
@@
 F 0 "C31" H 7790 2171 50  0000 L CNN
 F 1 ".1u" H 7790 2080 50  0000 L CNN
-F 2 "" H 7713 1975 50  0001 C CNN
+F 2 "Capacitor_SMD:C_0603_1608Metric" H 7713 1975 50  0001 C CNN
 F 3 "~" H 7675 2125 50  0001 C CNN
 	1    7675 2125
@@
 F 0 "C32" H 8115 2171 50  0000 L CNN
 F 1 "10u" H 8115 2080 50  0000 L CNN
-F 2 "" H 8038 1975 50  0001 C CNN
+F 2 "Capacitor_SMD:C_0603_1608Metric" H 8038 1975 50  0001 C CNN
 F 3 "~" H 8000 2125 50  0001 C CNN
 	1    8000 2125
@@
 F 0 "R36" H 8545 2146 50  0000 L CNN
 F 1 "10k" H 8545 2055 50  0000 L CNN
-F 2 "" V 8405 2100 50  0001 C CNN
+F 2 "Resistor_SMD:R_0603_1608Metric" V 8405 2100 50  0001 C CNN
 F 3 "~" H 8475 2100 50  0001 C CNN
 	1    8475 2100
@@
 F 0 "C33" H 8890 2546 50  0000 L CNN
 F 1 ".1u" H 8890 2455 50  0000 L CNN
-F 2 "" H 8813 2350 50  0001 C CNN
+F 2 "Capacitor_SMD:C_0603_1608Metric" H 8813 2350 50  0001 C CNN
 F 3 "~" H 8775 2500 50  0001 C CNN
 	1    8775 2500
@@
 F 0 "SW4" V 9154 2598 50  0000 L CNN
 F 1 "BOOT" V 9245 2598 50  0000 L CNN
-F 2 "" H 9200 2650 50  0001 C CNN
+F 2 "Button_Switch_SMD:SW_SPST_EVQQ2" H 9200 2650 50  0001 C CNN
 F 3 "~" H 9200 2650 50  0001 C CNN
 	1    9200 2450
@@
 F 0 "D3" H 8668 3070 50  0000 C CNN
 F 1 "LED" H 8668 3161 50  0000 C CNN
-F 2 "" H 8675 3325 50  0001 C CNN
+F 2 "LED_SMD:LED_0603_1608Metric_Castellated" H 8675 3325 50  0001 C CNN
 F 3 "~" H 8675 3325 50  0001 C CNN
 	1    8675 3325
@@
 F 0 "R35" V 8557 3325 50  0000 C CNN
 F 1 "100" V 8466 3325 50  0000 C CNN
-F 2 "" V 8280 3325 50  0001 C CNN
+F 2 "Resistor_SMD:R_0603_1608Metric" V 8280 3325 50  0001 C CNN
 F 3 "~" H 8350 3325 50  0001 C CNN
 	1    8350 3325
@@
 F 0 "R34" H 6545 2446 50  0000 L CNN
 F 1 "R" H 6545 2355 50  0000 L CNN
-F 2 "" V 6405 2400 50  0001 C CNN
+F 2 "Resistor_SMD:R_0603_1608Metric" V 6405 2400 50  0001 C CNN
 F 3 "~" H 6475 2400 50  0001 C CNN
 	1    6475 2400
@@
 F 0 "C30" H 5925 2925 50  0000 L CNN
 F 1 ".1u" H 5925 2750 50  0000 L CNN
-F 2 "" H 6113 2700 50  0001 C CNN
+F 2 "Capacitor_SMD:C_0603_1608Metric" H 6113 2700 50  0001 C CNN
 F 3 "~" H 6075 2850 50  0001 C CNN
 	1    6075 2850

Commit message: cam and more...
Parts:
- J5: footprint (none) -> Connector_PinSocket_1.27mm:PinSocket_1x03_P1.27mm_Vertical_SMD_Pin1Left
Changed lines of the file:
@@
 F 0 "J5" H 8858 5306 50  0000 C CNN
 F 1 "Conn_01x03_Male" H 8858 5215 50  0000 C CNN
-F 2 "" H 8750 5025 50  0001 C CNN
+F 2 "Connector_PinSocket_1.27mm:PinSocket_1x03_P1.27mm_Vertical_SMD_Pin1Left" H 8750 5025 50  0001 C CNN
 F 3 "~" H 8750 5025 50  0001 C CNN
 	1    8750 5025
