File: prius_gen2_kicad/powersupply.sch (KiCad schematic (older format))
At the start: 20 parts

Commit message: fixed ERC
Parts:
- gave numbers to parts that had none: 20
Changed lines of the file:
@@
 $EndDescr
 $Comp
-L Regulator_Linear:AZ1117-3.3 U?
+L Regulator_Linear:AZ1117-3.3 U8
 U 1 1 60E19B1F
 P 9250 3500
-F 0 "U?" H 9250 3742 50  0000 C CNN
+F 0 "U8" H 9250 3742 50  0000 C CNN
 F 1 "AZ1117-3.3" H 9250 3651 50  0000 C CNN
 F 2 "" H 9250 3750 50  0001 C CIN
@@
 $EndComp
 $Comp
-L Device:D_Schottky D?
+L Device:D_Schottky D5
 U 1 1 60E1C178
 P 2600 3250
-F 0 "D?" H 2600 3033 50  0000 C CNN
+F 0 "D5" H 2600 3033 50  0000 C CNN
 F 1 "D_Schottky" H 2600 3124 50  0000 C CNN
 F 2 "" H 2600 3250 50  0001 C CNN
@@
 $EndComp
 $Comp
-L Diode:ESD9B3.3ST5G D?
+L Diode:ESD9B3.3ST5G D4
 U 1 1 60E1E16A
 P 2000 3500
-F 0 "D?" V 1954 3579 50  0000 L CNN
+F 0 "D4" V 1954 3579 50  0000 L CNN
 F 1 "SM15T33CA" V 2045 3579 50  0000 L CNN
 F 2 "Diode_SMD:D_SOD-923" H 2000 3500 50  0001 C CNN
@@
 $EndComp
 $Comp
-L power:GND #PWR?
+L power:GND #PWR0159
 U 1 1 60E1E77D
 P 2000 3800
-F 0 "#PWR?" H 2000 3550 50  0001 C CNN
+F 0 "#PWR0159" H 2000 3550 50  0001 C CNN
 F 1 "GND" H 2005 3627 50  0000 C CNN
 F 2 "" H 2000 3800 50  0001 C CNN
@@
 $EndComp
 $Comp
-L lmr14020:LMR14020 U?
+L lmr14020:LMR14020 U7
 U 1 1 60E1F8E0
 P 5725 3450
-F 0 "U?" H 5825 3875 50  0000 C CNN
+F 0 "U7" H 5825 3875 50  0000 C CNN
 F 1 "LMR14020" H 5825 3784 50  0000 C CNN
 F 2 "" H 5725 3450 50  0001 C CNN
@@
 $EndComp
 $Comp
-L Device:R R?
+L Device:R R37
 U 1 1 60E21BB5
 P 3025 3450
-F 0 "R?" H 3095 3496 50  0000 L CNN
+F 0 "R37" H 3095 3496 50  0000 L CNN
 F 1 "1" H 3095 3405 50  0000 L CNN
 F 2 "" V 2955 3450 50  0001 C CNN
@@
 $EndComp
 $Comp
-L Device:C C?
+L Device:C C34
 U 1 1 60E2218B
 P 3025 3900
-F 0 "C?" H 3140 3946 50  0000 L CNN
+F 0 "C34" H 3140 3946 50  0000 L CNN
 F 1 "4.7uF" H 3140 3855 50  0000 L CNN
 F 2 "" H 3063 3750 50  0001 C CNN
@@
 $EndComp
 $Comp
-L pspice:INDUCTOR L?
+L pspice:INDUCTOR L1
 U 1 1 60E228C0
 P 3600 3250
-F 0 "L?" H 3600 3465 50  0000 C CNN
+F 0 "L1" H 3600 3465 50  0000 C CNN
 F 1 "2.2uH" H 3600 3374 50  0000 C CNN
 F 2 "" H 3600 3250 50  0001 C CNN
@@
 $EndComp
 $Comp
-L Device:CP C?
+L Device:CP C35
 U 1 1 60E23CAA
 P 4100 3525
-F 0 "C?" H 4218 3571 50  0000 L CNN
+F 0 "C35" H 4218 3571 50  0000 L CNN
 F 1 "56uF" H 4218 3480 50  0000 L CNN
 F 2 "" H 4138 3375 50  0001 C CNN
@@
 $EndComp
 $Comp
-L Device:C C?
+L Device:C C36
 U 1 1 60E24302
 P 4575 3525
-F 0 "C?" H 4690 3571 50  0000 L CNN
+F 0 "C36" H 4690 3571 50  0000 L CNN
 F 1 "1uF" H 4690 3480 50  0000 L CNN
 F 2 "" H 4613 3375 50  0001 C CNN
@@
 	3850 3250 4100 3250
 $Comp
-L power:GND #PWR?
+L power:GND #PWR0160
 U 1 1 60E2C117
 P 3025 4150
-F 0 "#PWR?" H 3025 3900 50  0001 C CNN
+F 0 "#PWR0160" H 3025 3900 50  0001 C CNN
 F 1 "GND" H 3030 3977 50  0000 C CNN
 F 2 "" H 3025 4150 50  0001 C CNN
@@
 $EndComp
 $Comp
-L power:GND #PWR?
+L power:GND #PWR0161
 U 1 1 60E2C381
 P 4100 3800
-F 0 "#PWR?" H 4100 3550 50  0001 C CNN
+F 0 "#PWR0161" H 4100 3550 50  0001 C CNN
 F 1 "GND" H 4105 3627 50  0000 C CNN
 F 2 "" H 4100 3800 50  0001 C CNN
@@
 $EndComp
 $Comp
-L power:GND #PWR?
+L power:GND #PWR0162
 U 1 1 60E2C5C8
 P 4575 3800
-F 0 "#PWR?" H 4575 3550 50  0001 C CNN
+F 0 "#PWR0162" H 4575 3550 50  0001 C CNN
 F 1 "GND" H 4580 3627 50  0000 C CNN
 F 2 "" H 4575 3800 50  0001 C CNN
@@
 Wire Wire Line
 	5050 3400 5050 3250
-Connection ~ 5050 3250
-Wire Wire Line
-	5050 3250 5425 3250
-$Comp
-L Device:R R?
+$Comp
+L Device:R R38
 U 1 1 60E30342
 P 5025 3800
-F 0 "R?" H 5095 3846 50  0000 L CNN
+F 0 "R38" H 5095 3846 50  0000 L CNN
 F 1 "10k" H 5095 3755 50  0000 L CNN
 F 2 "" V 4955 3800 50  0001 C CNN
@@
 $EndComp
 $Comp
-L power:GND #PWR?
+L power:GND #PWR0163
 U 1 1 60E3058E
 P 5025 4050
-F 0 "#PWR?" H 5025 3800 50  0001 C CNN
+F 0 "#PWR0163" H 5025 3800 50  0001 C CNN
 F 1 "GND" H 5030 3877 50  0000 C CNN
 F 2 "" H 5025 4050 50  0001 C CNN
@@
 	5025 3650 5025 3550
 $Comp
-L Device:C C?
+L Device:C C37
 U 1 1 60E311D9
 P 5350 3975
-F 0 "C?" H 5465 4021 50  0000 L CNN
+F 0 "C37" H 5465 4021 50  0000 L CNN
 F 1 "10nF" H 5465 3930 50  0000 L CNN
 F 2 "" H 5388 3825 50  0001 C CNN
@@
 $EndComp
 $Comp
-L power:GND #PWR?
+L power:GND #PWR0164
 U 1 1 60E316F6
 P 5350 4250
-F 0 "#PWR?" H 5350 4000 50  0001 C CNN
+F 0 "#PWR0164" H 5350 4000 50  0001 C CNN
 F 1 "GND" H 5355 4077 50  0000 C CNN
 F 2 "" H 5350 4250 50  0001 C CNN
@@
 	5350 3825 5350 3750
 $Comp
-L power:GND #PWR?
+L power:GND #PWR0165
 U 1 1 60E327B6
 P 5825 4025
-F 0 "#PWR?" H 5825 3775 50  0001 C CNN
+F 0 "#PWR0165" H 5825 3775 50  0001 C CNN
 F 1 "GND" H 5830 3852 50  0000 C CNN
 F 2 "" H 5825 4025 50  0001 C CNN
@@
 Connection ~ 5825 3975
 $Comp
-L Device:C C?
+L Device:C C38
 U 1 1 60E384EC
 P 6525 3225
-F 0 "C?" H 6640 3271 50  0000 L CNN
+F 0 "C38" H 6640 3271 50  0000 L CNN
 F 1 "100nF" H 6640 3180 50  0000 L CNN
 F 2 "" H 6563 3075 50  0001 C CNN
@@
 	6525 3000 6525 3075
 $Comp
-L Device:D_Schottky D?
+L Device:D_Schottky D6
 U 1 1 60E3A3D8
 P 7050 3225
-F 0 "D?" V 7096 3145 50  0000 R CNN
+F 0 "D6" V 7096 3145 50  0000 R CNN
 F 1 "D_Schottky" V 7005 3145 50  0000 R CNN
 F 2 "" H 7050 3225 50  0001 C CNN
@@
 $EndComp
 $Comp
-L pspice:INDUCTOR L?
+L pspice:INDUCTOR L2
 U 1 1 60E3ADD5
 P 7450 3500
-F 0 "L?" H 7450 3715 50  0000 C CNN
+F 0 "L2" H 7450 3715 50  0000 C CNN
 F 1 "INDUCTOR" H 7450 3624 50  0000 C CNN
 F 2 "" H 7450 3500 50  0001 C CNN
@@
 	7050 3500 7200 3500
 $Comp
-L power:GND #PWR?
+L power:GND #PWR0166
 U 1 1 60E3CF68
 P 7050 3025
-F 0 "#PWR?" H 7050 2775 50  0001 C CNN
+F 0 "#PWR0166" H 7050 2775 50  0001 C CNN
 F 1 "GND" H 7055 2852 50  0000 C CNN
 F 2 "" H 7050 3025 50  0001 C CNN
@@
 	7050 3025 7050 3075
 $Comp
-L Device:R R?
+L Device:R R39
 U 1 1 60E417F0
 P 6400 3975
-F 0 "R?" H 6470 4021 50  0000 L CNN
+F 0 "R39" H 6470 4021 50  0000 L CNN
 F 1 "12k" H 6470 3930 50  0000 L CNN
 F 2 "" V 6330 3975 50  0001 C CNN
@@
 $EndComp
 $Comp
-L Device:R R?
+L Device:R R40
 U 1 1 60E41BDB
 P 6900 3750
-F 0 "R?" V 6693 3750 50  0000 C CNN
+F 0 "R40" V 6693 3750 50  0000 C CNN
 F 1 "68k" V 6784 3750 50  0000 C CNN
 F 2 "" V 6830 3750 50  0001 C CNN
@@
 	6400 3750 6225 3750
 $Comp
-L power:GND #PWR?
+L power:GND #PWR0167
 U 1 1 60E4322F
 P 6400 4250
-F 0 "#PWR?" H 6400 4000 50  0001 C CNN
+F 0 "#PWR0167" H 6400 4000 50  0001 C CNN
 F 1 "GND" H 6405 4077 50  0000 C CNN
 F 2 "" H 6400 4250 50  0001 C CNN
@@
 	6400 4250 6400 4125
 $Comp
-L Device:C C?
+L Device:C C39
 U 1 1 60E4437D
 P 6900 4000
-F 0 "C?" V 6675 4000 50  0000 C CNN
+F 0 "C39" V 6675 4000 50  0000 C CNN
 F 1 "330pF" V 6750 4000 50  0000 C CNN
 F 2 "" H 6938 3850 50  0001 C CNN
@@
 	6675 3750 6400 3750
 $Comp
-L Device:C C?
+L Device:C C40
 U 1 1 60E4C1B8
 P 8125 3725
-F 0 "C?" H 8240 3771 50  0000 L CNN
+F 0 "C40" H 8240 3771 50  0000 L CNN
 F 1 "10uF" H 8240 3680 50  0000 L CNN
 F 2 "" H 8163 3575 50  0001 C CNN
@@
 	7150 3750 7800 3750
 $Comp
-L power:GND #PWR?
+L power:GND #PWR0168
 U 1 1 60E4E5F9
 P 8125 3975
-F 0 "#PWR?" H 8125 3725 50  0001 C CNN
+F 0 "#PWR0168" H 8125 3725 50  0001 C CNN
 F 1 "GND" H 8130 3802 50  0000 C CNN
 F 2 "" H 8125 3975 50  0001 C CNN
@@
 	8125 3975 8125 3875
 $Comp
-L Device:C C?
+L Device:C C41
 U 1 1 60E50974
 P 8575 3725
-F 0 "C?" H 8690 3771 50  0000 L CNN
+F 0 "C41" H 8690 3771 50  0000 L CNN
 F 1 "10uF" H 8690 3680 50  0000 L CNN
 F 2 "" H 8613 3575 50  0001 C CNN
@@
 $EndComp
 $Comp
-L power:GND #PWR?
+L power:GND #PWR0169
 U 1 1 60E5097A
 P 8575 3975
-F 0 "#PWR?" H 8575 3725 50  0001 C CNN
+F 0 "#PWR0169" H 8575 3725 50  0001 C CNN
 F 1 "GND" H 8580 3802 50  0000 C CNN
 F 2 "" H 8575 3975 50  0001 C CNN
@@
 Connection ~ 8575 3500
 $Comp
-L power:GND #PWR?
+L power:GND #PWR0170
 U 1 1 60E55CFA
 P 9250 3975
-F 0 "#PWR?" H 9250 3725 50  0001 C CNN
+F 0 "#PWR0170" H 9250 3725 50  0001 C CNN
 F 1 "GND" H 9255 3802 50  0000 C CNN
 F 2 "" H 9250 3975 50  0001 C CNN
@@
 	9250 3975 9250 3800
 $Comp
-L power:+3V3 #PWR?
+L power:+3V3 #PWR0171
 U 1 1 60E57207
 P 9875 3350
-F 0 "#PWR?" H 9875 3200 50  0001 C CNN
+F 0 "#PWR0171" H 9875 3200 50  0001 C CNN
 F 1 "+3V3" H 9890 3523 50  0000 C CNN
 F 2 "" H 9875 3350 50  0001 C CNN
@@
 $EndComp
 $Comp
-L power:GND #PWR?
+L power:GND #PWR0172
 U 1 1 60E57682
 P 9875 3975
-F 0 "#PWR?" H 9875 3725 50  0001 C CNN
+F 0 "#PWR0172" H 9875 3725 50  0001 C CNN
 F 1 "GND" H 9880 3802 50  0000 C CNN
 F 2 "" H 9875 3975 50  0001 C CNN
@@
 	9875 3575 9875 3500
 $Comp
-L Device:C C?
+L Device:C C42
 U 1 1 60E57387
 P 9875 3725
-F 0 "C?" H 9990 3771 50  0000 L CNN
+F 0 "C42" H 9990 3771 50  0000 L CNN
 F 1 "4.7uF" H 9990 3680 50  0000 L CNN
 F 2 "" H 9913 3575 50  0001 C CNN
@@
 	9875 3500 9875 3350
 $Comp
-L power:PWR_FLAG #FLG?
+L power:PWR_FLAG #FLG0101
 U 1 1 60E727E5
 P 2150 3250
-F 0 "#FLG?" H 2150 3325 50  0001 C CNN
+F 0 "#FLG0101" H 2150 3325 50  0001 C CNN
 F 1 "PWR_FLAG" H 2150 3423 50  0000 C CNN
 F 2 "" H 2150 3250 50  0001 C CNN
@@
 	2150 3250 2450 3250
 $Comp
-L power:PWR_FLAG #FLG?
+L power:PWR_FLAG #FLG0102
 U 1 1 60E72D3D
 P 8125 3500
-F 0 "#FLG?" H 8125 3575 50  0001 C CNN
+F 0 "#FLG0102" H 8125 3575 50  0001 C CNN
 F 1 "PWR_FLAG" H 8125 3673 50  0000 C CNN
 F 2 "" H 8125 3500 50  0001 C CNN
@@
 $EndComp
 $Comp
-L power:+5V #PWR?
+L power:+5V #PWR0173
 U 1 1 60E7481E
 P 8575 3350
-F 0 "#PWR?" H 8575 3200 50  0001 C CNN
+F 0 "#PWR0173" H 8575 3200 50  0001 C CNN
 F 1 "+5V" H 8590 3523 50  0000 C CNN
 F 2 "" H 8575 3350 50  0001 C CNN
@@
 	8575 3350 8575 3500
 $Comp
-L power:+12V #PWR?
+L power:+12V #PWR0174
 U 1 1 60FDA2CE
 P 1550 3150
-F 0 "#PWR?" H 1550 3000 50  0001 C CNN
+F 0 "#PWR0174" H 1550 3000 50  0001 C CNN
 F 1 "+12V" H 1565 3323 50  0000 C CNN
 F 2 "" H 1550 3150 50  0001 C CNN
@@
 Text Notes 8850 3050 0    50   ~ 0
 3.3V
+Wire Wire Line
+	5425 3250 5250 3250
+Connection ~ 5050 3250
+$Comp
+L power:PWR_FLAG #FLG0103
+U 1 1 61AB96E0
+P 5250 3250
+F 0 "#FLG0103" H 5250 3325 50  0001 C CNN
+F 1 "PWR_FLAG" H 5250 3423 50  0000 C CNN
+F 2 "" H 5250 3250 50  0001 C CNN
+F 3 "~" H 5250 3250 50  0001 C CNN
+	1    5250 3250
+	1    0    0    -1
+$EndComp
+Connection ~ 5250 3250
+Wire Wire Line
+	5250 3250 5050 3250
 $EndSCHEMATC

Commit message: started routing
Parts:
- C34, C36, C37, C38, C39, C40, C41, C42: footprint (none) -> Capacitor_SMD:C_0603_1608Metric
- C35: footprint (none) -> Capacitor_THT:CP_Radial_D8.0mm_P3.50mm
- D4: footprint Diode_SMD:D_SOD-923 -> Diode_SMD:D_SMC
- D5, D6: footprint (none) -> Diode_SMD:D_SMA
- L1: footprint (none) -> Inductor_SMD:L_1210_3225Metric
- L2: value INDUCTOR -> 10u
- R37, R38, R39, R40: footprint (none) -> Resistor_SMD:R_0603_1608Metric
- U7: footprint (none) -> Package_SO:SOIC-8-1EP_3.9x4.9mm_P1.27mm_EP2.29x3mm
- U8: footprint (none) -> Package_TO_SOT_SMD:SOT-223-3_TabPin2
Changed lines of the file:
@@
 F 0 "U8" H 9250 3742 50  0000 C CNN
 F 1 "AZ1117-3.3" H 9250 3651 50  0000 C CNN
-F 2 "" H 9250 3750 50  0001 C CIN
+F 2 "Package_TO_SOT_SMD:SOT-223-3_TabPin2" H 9250 3750 50  0001 C CIN
 F 3 "https://www.diodes.com/assets/Datasheets/AZ1117.pdf" H 9250 3500 50  0001 C CNN
 	1    9250 3500
@@
 F 0 "D5" H 2600 3033 50  0000 C CNN
 F 1 "D_Schottky" H 2600 3124 50  0000 C CNN
-F 2 "" H 2600 3250 50  0001 C CNN
+F 2 "Diode_SMD:D_SMA" H 2600 3250 50  0001 C CNN
 F 3 "~" H 2600 3250 50  0001 C CNN
 	1    2600 3250
@@
 F 0 "D4" V 1954 3579 50  0000 L CNN
 F 1 "SM15T33CA" V 2045 3579 50  0000 L CNN
-F 2 "Diode_SMD:D_SOD-923" H 2000 3500 50  0001 C CNN
+F 2 "Diode_SMD:D_SMC" H 2000 3500 50  0001 C CNN
 F 3 "https://www.onsemi.com/pub/Collateral/ESD9B-D.PDF" H 2000 3500 50  0001 C CNN
 	1    2000 3500
@@
 F 0 "U7" H 5825 3875 50  0000 C CNN
 F 1 "LMR14020" H 5825 3784 50  0000 C CNN
-F 2 "" H 5725 3450 50  0001 C CNN
+F 2 "Package_SO:SOIC-8-1EP_3.9x4.9mm_P1.27mm_EP2.29x3mm" H 5725 3450 50  0001 C CNN
 F 3 "" H 5725 3450 50  0001 C CNN
 	1    5725 3450
@@
 F 0 "R37" H 3095 3496 50  0000 L CNN
 F 1 "1" H 3095 3405 50  0000 L CNN
-F 2 "" V 2955 3450 50  0001 C CNN
+F 2 "Resistor_SMD:R_0603_1608Metric" V 2955 3450 50  0001 C CNN
 F 3 "~" H 3025 3450 50  0001 C CNN
 	1    3025 3450
@@
 F 0 "C34" H 3140 3946 50  0000 L CNN
 F 1 "4.7uF" H 3140 3855 50  0000 L CNN
-F 2 "" H 3063 3750 50  0001 C CNN
+F 2 "Capacitor_SMD:C_0603_1608Metric" H 3063 3750 50  0001 C CNN
 F 3 "~" H 3025 3900 50  0001 C CNN
 	1    3025 3900
@@
 F 0 "L1" H 3600 3465 50  0000 C CNN
 F 1 "2.2uH" H 3600 3374 50  0000 C CNN
-F 2 "" H 3600 3250 50  0001 C CNN
+F 2 "Inductor_SMD:L_1210_3225Metric" H 3600 3250 50  0001 C CNN
 F 3 "~" H 3600 3250 50  0001 C CNN
 	1    3600 3250
@@
 F 0 "C35" H 4218 3571 50  0000 L CNN
 F 1 "56uF" H 4218 3480 50  0000 L CNN
-F 2 "" H 4138 3375 50  0001 C CNN
+F 2 "Capacitor_THT:CP_Radial_D8.0mm_P3.50mm" H 4138 3375 50  0001 C CNN
 F 3 "~" H 4100 3525 50  0001 C CNN
 	1    4100 3525
@@
 F 0 "C36" H 4690 3571 50  0000 L CNN
 F 1 "1uF" H 4690 3480 50  0000 L CNN
-F 2 "" H 4613 3375 50  0001 C CNN
+F 2 "Capacitor_SMD:C_0603_1608Metric" H 4613 3375 50  0001 C CNN
 F 3 "~" H 4575 3525 50  0001 C CNN
 	1    4575 3525
@@
 F 0 "R38" H 5095 3846 50  0000 L CNN
 F 1 "10k" H 5095 3755 50  0000 L CNN
-F 2 "" V 4955 3800 50  0001 C CNN
+F 2 "Resistor_SMD:R_0603_1608Metric" V 4955 3800 50  0001 C CNN
 F 3 "~" H 5025 3800 50  0001 C CNN
 	1    5025 3800
@@
 F 0 "C37" H 5465 4021 50  0000 L CNN
 F 1 "10nF" H 5465 3930 50  0000 L CNN
-F 2 "" H 5388 3825 50  0001 C CNN
+F 2 "Capacitor_SMD:C_0603_1608Metric" H 5388 3825 50  0001 C CNN
 F 3 "~" H 5350 3975 50  0001 C CNN
 	1    5350 3975
@@
 F 0 "C38" H 6640 3271 50  0000 L CNN
 F 1 "100nF" H 6640 3180 50  0000 L CNN
-F 2 "" H 6563 3075 50  0001 C CNN
+F 2 "Capacitor_SMD:C_0603_1608Metric" H 6563 3075 50  0001 C CNN
 F 3 "~" H 6525 3225 50  0001 C CNN
 	1    6525 3225
@@
 F 0 "D6" V 7096 3145 50  0000 R CNN
 F 1 "D_Schottky" V 7005 3145 50  0000 R CNN
-F 2 "" H 7050 3225 50  0001 C CNN
+F 2 "Diode_SMD:D_SMA" H 7050 3225 50  0001 C CNN
 F 3 "~" H 7050 3225 50  0001 C CNN
 	1    7050 3225
@@
 P 7450 3500
 F 0 "L2" H 7450 3715 50  0000 C CNN
-F 1 "INDUCTOR" H 7450 3624 50  0000 C CNN
+F 1 "10u" H 7450 3624 50  0000 C CNN
 F 2 "" H 7450 3500 50  0001 C CNN
 F 3 "~" H 7450 3500 50  0001 C CNN
@@
 F 0 "R39" H 6470 4021 50  0000 L CNN
 F 1 "12k" H 6470 3930 50  0000 L CNN
-F 2 "" V 6330 3975 50  0001 C CNN
+F 2 "Resistor_SMD:R_0603_1608Metric" V 6330 3975 50  0001 C CNN
 F 3 "~" H 6400 3975 50  0001 C CNN
 	1    6400 3975
@@
 F 0 "R40" V 6693 3750 50  0000 C CNN
 F 1 "68k" V 6784 3750 50  0000 C CNN
-F 2 "" V 6830 3750 50  0001 C CNN
+F 2 "Resistor_SMD:R_0603_1608Metric" V 6830 3750 50  0001 C CNN
 F 3 "~" H 6900 3750 50  0001 C CNN
 	1    6900 3750
@@
 F 0 "C39" V 6675 4000 50  0000 C CNN
 F 1 "330pF" V 6750 4000 50  0000 C CNN
-F 2 "" H 6938 3850 50  0001 C CNN
+F 2 "Capacitor_SMD:C_0603_1608Metric" H 6938 3850 50  0001 C CNN
 F 3 "~" H 6900 4000 50  0001 C CNN
 	1    6900 4000
@@
 F 0 "C40" H 8240 3771 50  0000 L CNN
 F 1 "10uF" H 8240 3680 50  0000 L CNN
-F 2 "" H 8163 3575 50  0001 C CNN
+F 2 "Capacitor_SMD:C_0603_1608Metric" H 8163 3575 50  0001 C CNN
 F 3 "~" H 8125 3725 50  0001 C CNN
 	1    8125 3725
@@
 F 0 "C41" H 8690 3771 50  0000 L CNN
 F 1 "10uF" H 8690 3680 50  0000 L CNN
-F 2 "" H 8613 3575 50  0001 C CNN
+F 2 "Capacitor_SMD:C_0603_1608Metric" H 8613 3575 50  0001 C CNN
 F 3 "~" H 8575 3725 50  0001 C CNN
 	1    8575 3725
@@
 F 0 "C42" H 9990 3771 50  0000 L CNN
 F 1 "4.7uF" H 9990 3680 50  0000 L CNN
-F 2 "" H 9913 3575 50  0001 C CNN
+F 2 "Capacitor_SMD:C_0603_1608Metric" H 9913 3575 50  0001 C CNN
 F 3 "~" H 9875 3725 50  0001 C CNN
 	1    9875 3725

Commit message: cam and more...
Parts:
- L2: footprint (none) -> prius_gen2_kicad:MWSA0503
Changed lines of the file:
@@
 F 0 "L2" H 7450 3715 50  0000 C CNN
 F 1 "10u" H 7450 3624 50  0000 C CNN
-F 2 "" H 7450 3500 50  0001 C CNN
+F 2 "prius_gen2_kicad:MWSA0503" H 7450 3500 50  0001 C CNN
 F 3 "~" H 7450 3500 50  0001 C CNN
 	1    7450 3500
