File: prius_gen2_kicad/prius_gen2.kicad_pcb (KiCad board)
At the start: 2 copper layers, 147.8 x 65 mm, 140 parts, among them J1 Conn_02x05_Odd_Even, J2 Conn_01x06, J3 Conn_01x23, J4 Conn_01x14, Q1 IRLZ14SPBF, Q2 IRLZ14SPBF, SW1 SW_Push, SW2 SW_Push, SW3 RESET, SW4 BOOT, U1 STM32F103RBTx, U2 MCP602, U3 ULN2003A, U4 TDA2822D, U5 TJA1051T-3, U6 ESP32-WROOM-32, U7 LMR14020, U8 AZ1117-3.3, Y1 8MHz

Commit message: cam and more...
Parts:
- added G***: LOGO, prius_gen2_kicad:rsspeed, B.Cu at (138.5, 94.7)
- added L2: 10u, prius_gen2_kicad:MWSA0503, F.Cu at (139.3, 118.3)
- C21, C35, J1, J2: moved to B.Cu
- moved C21 15.1 mm to (139.2, 123.4), turned to 270 degrees
- moved C4 9.75 mm to (141.7, 68.0), turned to 90 degrees
- moved R1 9.28 mm to (141.7, 71.4), turned to 90 degrees
- moved J2 1.34 mm to (136.8, 69.7), turned to 270 degrees
- moved R43 0.20 mm to (115.1, 87.8)
- moved R44 0.20 mm to (115.1, 89.5)
Routing:
- net +5V: track 21.3 -> 358.9 mm, vias 0 -> 13
- net +3V3: track 40.7 -> 286.3 mm, vias 0 -> 16
- net /nRESET: track 0.00 -> 81.3 mm, vias 0 -> 4
- net /ADC13: track 0.00 -> 77.9 mm, vias 0 -> 4
- net /ADC12: track 6.66 -> 83.1 mm, vias 0 -> 4
- net /ADC11: track 6.66 -> 80.2 mm, vias 0 -> 2
- net /ADC10: track 6.66 -> 77.1 mm, vias 0 -> 2
- net /ADC9: track 0.00 -> 69.7 mm, vias 0 -> 4
- net Net-(J4-Pad10): track 0.00 -> 57.2 mm, vias 0 -> 1
- net Net-(J4-Pad11): track 0.00 -> 54.1 mm, vias 0 -> 1
- net /TIM3_ETR: track 0.00 -> 50.7 mm, vias 0 -> 2
- net /CAN_TX: track 0.00 -> 49.0 mm, vias 0 -> 2
- net /ADC14: track 0.00 -> 49.0 mm, vias 0 -> 6
- net /Connectors/GIWA: track 0.00 -> 48.9 mm, vias 0 -> 1
- net /CAN_RX: track 0.00 -> 46.9 mm, vias 0 -> 2
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- added copper zone on B.Cu, net GND
- added copper zone on F.Cu, net GND
Other:
- board text added: "+12V"
- board text added: "+5V"
- board text added: "BOOT"
- board text added: "BRK"
- board text added: "CAN"
- board text added: "CANH"
- board text added: "CANL"
- board text added: "CPWM"
- board text added: "DAR"
- board text added: "DCSW"
- board text added: "ENC"
- board text added: "ENCA"
- board text added: "ENCB"
- board text added: "ESP"
- board text added: "FIL"
- board text added: "FWD"
- board text added: "GIVA"
- board text added: "GIWA"
- board text added: "GND"
- board text added: "LVL"
- board text added: "MFIV"
- board text added: "MIVA"
- board text added: "MIVT"
- board text added: "MIWA"
- board text added: "MTP+"
- board text added: "MTP-"
- board text added: "MUU"
- board text added: "MVU"
- board text added: "MWU"
- board text added: "PRE"
- board text added: "PSU"
- board text added: "Prius G2 rev 1 2021-07"
- board text added: "R1"
- board text added: "R2"
- board text added: "RES"
- board text added: "REV"
- board text added: "RST"
- board text added: "START"
- board text added: "SWD"
- board text added: "TH1"
- board text added: "TH2"
- board text added: "VH"
- board text added: "powered by openinverter.org"
