File: prius_gen2_kicad/prius_gen2.sch (KiCad schematic (older format))
At the start: 18 parts

Commit message: more schematics
Parts:
- removed J?: Conn_02x03_Odd_Even, symbol Connector_Generic:Conn_02x03_Odd_Even
- added J?: Conn_02x05_Odd_Even, symbol Connector_Generic:Conn_02x05_Odd_Even
- added J?: Conn_01x06, symbol Connector_Generic:Conn_01x06
Connections:
- net +3V3: now also J?.1 (Pin_1), J?.1 (Pin_1)
- net GND: now also J?.3 (Pin_3), J?.5 (Pin_5), J?.5 (Pin_5), J?.9 (Pin_9)
- net SWCLK: now also J?.4 (Pin_4), J?.4 (Pin_4)
- net SWDIO: now also J?.2 (Pin_2), J?.2 (Pin_2)
- net NRST renamed nRST
- net nRST: now also J?.10 (Pin_10), J?.3 (Pin_3)
- no-connect marks 12 -> 16
Other:
- note added: "SWD DEBUG"
Changed lines of the file:
@@
 $Descr A4 11693 8268
 encoding utf-8
-Sheet 1 3
+Sheet 1 5
 Title ""
 Date ""
@@
 F 3 "http://www.st.com/st-web-ui/static/active/en/resource/technical/document/datasheet/CD00161566.pdf" H 5475 4125 50  0001 C CNN
 	1    5475 4125
-	1    0    0    -1
-$EndComp
-$Comp
-L Connector_Generic:Conn_02x03_Odd_Even J?
-U 1 1 60D26057
-P 8575 5600
-F 0 "J?" H 8625 5917 50  0000 C CNN
-F 1 "Conn_02x03_Odd_Even" H 8625 5826 50  0000 C CNN
-F 2 "" H 8575 5600 50  0001 C CNN
-F 3 "~" H 8575 5600 50  0001 C CNN
-	1    8575 5600
 	1    0    0    -1
 $EndComp
@@
 	4675 2725 4775 2725
 Text Label 4175 2525 0    50   ~ 0
-NRST
+nRST
 $Comp
 L power:GND #PWR?
@@
 	4675 2075 4675 2025
 Connection ~ 4325 2075
-Wire Wire Line
-	8375 5500 8075 5500
-Wire Wire Line
-	8075 5500 8075 5400
-$Comp
-L power:+3V3 #PWR?
-U 1 1 60DAD157
-P 8075 5400
-F 0 "#PWR?" H 8075 5250 50  0001 C CNN
-F 1 "+3V3" H 8090 5573 50  0000 C CNN
-F 2 "" H 8075 5400 50  0001 C CNN
-F 3 "" H 8075 5400 50  0001 C CNN
-	1    8075 5400
-	1    0    0    -1
-$EndComp
-$Comp
-L power:GND #PWR?
-U 1 1 60DAD95E
-P 8975 5750
-F 0 "#PWR?" H 8975 5500 50  0001 C CNN
-F 1 "GND" H 8980 5577 50  0000 C CNN
-F 2 "" H 8975 5750 50  0001 C CNN
-F 3 "" H 8975 5750 50  0001 C CNN
-	1    8975 5750
-	1    0    0    -1
-$EndComp
-Wire Wire Line
-	8975 5750 8975 5700
-Wire Wire Line
-	8975 5700 8875 5700
-Text Label 8075 5600 0    50   ~ 0
-SWDIO
-Wire Wire Line
-	8075 5600 8375 5600
-Text Label 8075 5700 0    50   ~ 0
-SWCLK
-Wire Wire Line
-	8075 5700 8375 5700
-Text Label 9175 5500 2    50   ~ 0
-NRST
-Wire Wire Line
-	9175 5500 8875 5500
 $Comp
 L Transistor_FET:IRLZ34N Q?
@@
 $EndSheet
 $Sheet
-S 8700 2825 1275 1750
+S 8075 2425 1275 1750
 U 611C056E
 F0 "Connectors" 50
 F1 "connectors.sch" 50
-F2 "ENC_B" I L 8700 3000 50
-F3 "ENC_A" I L 8700 2925 50
-F4 "R2" I L 8700 3275 50
-F5 "THROTTLE1" I L 8700 3375 50
-F6 "SIG_START" I L 8700 3475 50
-F7 "SIG_FWD" I L 8700 3575 50
-F8 "MTEMP-" I L 8700 3675 50
-F9 "OUT_DCSW" I L 8700 3775 50
-F10 "CAN_L" I R 9975 3050 50
-F11 "R1" I L 8700 3175 50
-F12 "THROTTLE2" I R 9975 3375 50
-F13 "SIG_BRAKE" I R 9975 3475 50
-F14 "SIG_REV" I R 9975 3575 50
-F15 "MTEMP+" I R 9975 3675 50
-F16 "OUT_PRE" I R 9975 3775 50
-F17 "CAN_H" I R 9975 2975 50
-F18 "GIVA" I R 9975 3875 50
-F19 "MIVA" I R 9975 3975 50
-F20 "GIWA" I R 9975 4075 50
-F21 "MIWA" I R 9975 4175 50
-F22 "VH" I R 9975 4275 50
-F23 "MFIV" I R 9975 4375 50
-F24 "MIVT" I R 9975 4475 50
-F25 "TIM1_CH2N" I L 8700 3875 50
-F26 "TIM1_CH3" I L 8700 3975 50
-F27 "TIM1_CH2" I L 8700 4075 50
-F28 "TIM1_CH1" I L 8700 4175 50
+F2 "ENC_B" I L 8075 2600 50
+F3 "ENC_A" I L 8075 2525 50
+F4 "R2" I L 8075 2875 50
+F5 "THROTTLE1" I L 8075 2975 50
+F6 "SIG_START" I L 8075 3075 50
+F7 "SIG_FWD" I L 8075 3175 50
+F8 "MTEMP-" I L 8075 3275 50
+F9 "OUT_DCSW" I L 8075 3375 50
+F10 "CAN_L" I R 9350 2650 50
+F11 "R1" I L 8075 2775 50
+F12 "THROTTLE2" I R 9350 2975 50
+F13 "SIG_BRAKE" I R 9350 3075 50
+F14 "SIG_REV" I R 9350 3175 50
+F15 "MTEMP+" I R 9350 3275 50
+F16 "OUT_PRE" I R 9350 3375 50
+F17 "CAN_H" I R 9350 2575 50
+F18 "GIVA" I R 9350 3475 50
+F19 "MIVA" I R 9350 3575 50
+F20 "GIWA" I R 9350 3675 50
+F21 "MIWA" I R 9350 3775 50
+F22 "VH" I R 9350 3875 50
+F23 "MFIV" I R 9350 3975 50
+F24 "MIVT" I R 9350 4075 50
+F25 "TIM1_CH2N" I L 8075 3475 50
+F26 "TIM1_CH3" I L 8075 3575 50
+F27 "TIM1_CH2" I L 8075 3675 50
+F28 "TIM1_CH1" I L 8075 3775 50
+$EndSheet
+Text Label 10975 4950 2    50   ~ 0
+SWDIO
+Text Label 10975 5050 2    50   ~ 0
+SWCLK
+Text Label 10975 5350 2    50   ~ 0
+nRST
+$Comp
+L power:GND #PWR?
+U 1 1 60E63029
+P 9925 6200
+F 0 "#PWR?" H 9925 5950 50  0001 C CNN
+F 1 "GND" H 9930 6027 50  0000 C CNN
+F 2 "" H 9925 6200 50  0001 C CNN
+F 3 "" H 9925 6200 50  0001 C CNN
+	1    9925 6200
+	1    0    0    -1
+$EndComp
+Wire Wire Line
+	9925 6200 9925 6100
+Wire Wire Line
+	9925 6100 10175 6100
+NoConn ~ 10175 6200
+Wire Wire Line
+	9900 6000 10175 6000
+Wire Wire Line
+	10175 5900 9900 5900
+Wire Wire Line
+	9900 5800 10175 5800
+Text Label 9900 6000 0    50   ~ 0
+SWCLK
+Text Label 9900 5900 0    50   ~ 0
+nRST
+Text Label 9900 5800 0    50   ~ 0
+SWDIO
+Wire Wire Line
+	10175 5700 10000 5700
+$Comp
+L power:+3V3 #PWR?
+U 1 1 60E4C8B5
+P 10000 5700
+F 0 "#PWR?" H 10000 5550 50  0001 C CNN
+F 1 "+3V3" H 10015 5873 50  0000 C CNN
+F 2 "" H 10000 5700 50  0001 C CNN
+F 3 "" H 10000 5700 50  0001 C CNN
+	1    10000 5700
+	0    -1   -1   0
+$EndComp
+NoConn ~ 10625 5150
+NoConn ~ 10625 5250
+Wire Wire Line
+	10975 5350 10625 5350
+Wire Wire Line
+	10625 5050 10975 5050
+Wire Wire Line
+	10975 4950 10625 4950
+NoConn ~ 10125 5250
+Wire Wire Line
+	9975 5150 9975 5350
+Connection ~ 9975 5150
+Wire Wire Line
+	10125 5150 9975 5150
+Connection ~ 9975 5350
+Wire Wire Line
+	9975 5050 9975 5150
+Wire Wire Line
+	10125 5050 9975 5050
+Wire Wire Line
+	9975 5350 9975 5375
+Wire Wire Line
+	10125 5350 9975 5350
+$Comp
+L power:GND #PWR?
+U 1 1 60E0BE1B
+P 9975 5375
+F 0 "#PWR?" H 9975 5125 50  0001 C CNN
+F 1 "GND" H 9980 5202 50  0000 C CNN
+F 2 "" H 9975 5375 50  0001 C CNN
+F 3 "" H 9975 5375 50  0001 C CNN
+	1    9975 5375
+	1    0    0    -1
+$EndComp
+Wire Wire Line
+	9975 4950 10125 4950
+$Comp
+L power:+3V3 #PWR?
+U 1 1 60E06F4A
+P 9975 4950
+F 0 "#PWR?" H 9975 4800 50  0001 C CNN
+F 1 "+3V3" H 9990 5123 50  0000 C CNN
+F 2 "" H 9975 4950 50  0001 C CNN
+F 3 "" H 9975 4950 50  0001 C CNN
+	1    9975 4950
+	0    -1   -1   0
+$EndComp
+$Comp
+L Connector_Generic:Conn_01x06 J?
+U 1 1 60E06842
+P 10375 5900
+F 0 "J?" H 10455 5892 50  0000 L CNN
+F 1 "Conn_01x06" H 10455 5801 50  0000 L CNN
+F 2 "" H 10375 5900 50  0001 C CNN
+F 3 "~" H 10375 5900 50  0001 C CNN
+	1    10375 5900
+	1    0    0    -1
+$EndComp
+$Comp
+L Connector_Generic:Conn_02x05_Odd_Even J?
+U 1 1 60E05B6A
+P 10325 5150
+F 0 "J?" H 10375 5567 50  0000 C CNN
+F 1 "Conn_02x05_Odd_Even" H 10375 5476 50  0000 C CNN
+F 2 "" H 10325 5150 50  0001 C CNN
+F 3 "~" H 10325 5150 50  0001 C CNN
+	1    10325 5150
+	1    0    0    -1
+$EndComp
+Wire Notes Line
+	9500 6525 9500 4525
+Wire Notes Line
+	9525 4525 11225 4525
+Text Notes 9550 4650 0    50   ~ 0
+SWD DEBUG
+$Sheet
+S 1650 4300 1225 500
+U 60EAB2A4
+F0 "Resolver" 50
+F1 "resolver.sch" 50
+$EndSheet
+$Sheet
+S 1700 5500 1200 450
+U 60EC424A
+F0 "Communication" 50
+F1 "communication.sch" 50
 $EndSheet
 $EndSCHEMATC

Commit message: schematics almost done
Parts:
- removed L?: 10uH, symbol Device:L
- added C? (x4): 10u, symbol Device:C
- added C?: 4.7u, symbol Device:C
- added FB?: Ferrite_Bead, symbol Device:Ferrite_Bead
- added R? (x2): 10k, symbol Device:R
- added SW? (x2): SW_Push, symbol Switch:SW_Push
- C? (x2): value 1uF -> 10n
- C? (x2): value 20pF -> 33p
- C? (x4): value 1uF -> 4.7u
- Y?: value Crystal -> 8MHz
Connections:
- net +3V3: now also C?.1, C?.1, C?.1, FB?.2, R?.1, SW?.1
- net GND: now also C?.2, C?.2, C?.2, C?.2, R?.2, SW?.1; no longer U?.60 (BOOT0)
- net TIM1_BKIN: now also U?.40 (PC9)
- net at C?.1, U?.13 (VDDA): now also C?.1, FB?.1
- net PC6 renamed REV
- net nRST renamed nRESET
- net nRESET: now also R?.2, SW?.2
- new net: R?.1, SW?.2, U?.60 (BOOT0)
Other:
- moved on the sheet: C?, D?, Q?, R?, U?, Y?

Commit message: fixed ERC
Parts:
- gave numbers to parts that had none: 28
Connections:
- net +3V3: now also C11.1
- net GND: now also C11.2
- net ADC15: no longer names the net of U1.25 (PC5)
- net TIM1_CH1N: no longer names the net of U1.34 (PB13)
- net TIM1_CH3N: no longer names the net of U1.36 (PB15)
- net TIM4_CH2: no longer names the net of U1.59 (PB7)
- net TIM4_CH3: no longer names the net of U1.61 (PB8)
- net TIM4_CH4: no longer names the net of U1.62 (PB9)
- no-connect marks 16 -> 22

Commit message: started routing
Parts:
- removed C11, C13, C9: 10u, symbol Device:C
- C1, C10, C12, C2, C3, C4, C5, C6, C7: footprint (none) -> Capacitor_SMD:C_0603_1608Metric
- C8: value 10u -> 4.7u; footprint (none) -> Capacitor_SMD:C_0603_1608Metric
- D1: footprint (none) -> LED_SMD:LED_0603_1608Metric_Castellated
- FB1: footprint (none) -> Capacitor_SMD:C_0805_2012Metric
- J1: footprint (none) -> Connector_PinHeader_1.27mm:PinHeader_2x05_P1.27mm_Vertical_SMD
- J2: footprint (none) -> Connector:Tag-Connect_TC2030-IDC-NL_2x03_P1.27mm_Vertical
- Q1, Q2: footprint Package_TO_SOT_THT:TO-220-3_Vertical -> Package_TO_SOT_SMD:TO-252-2
- R1, R2, R3, R4, R5: footprint (none) -> Resistor_SMD:R_0603_1608Metric
- SW1, SW2: footprint (none) -> Button_Switch_SMD:SW_SPST_EVQQ2
- Y1: footprint (none) -> Crystal:Crystal_SMD_5032-2Pin_5.0x3.2mm
Changed lines of the file:
@@
 F 0 "D1" H 3850 5375 50  0000 C CNN
 F 1 "LED" H 3725 5325 50  0000 C CNN
-F 2 "" H 3725 5450 50  0001 C CNN
+F 2 "LED_SMD:LED_0603_1608Metric_Castellated" H 3725 5450 50  0001 C CNN
 F 3 "~" H 3725 5450 50  0001 C CNN
 	1    3725 5450
@@
 F 0 "R2" V 3068 5450 50  0000 C CNN
 F 1 "680" V 3159 5450 50  0000 C CNN
-F 2 "" V 3205 5450 50  0001 C CNN
+F 2 "Resistor_SMD:R_0603_1608Metric" V 3205 5450 50  0001 C CNN
 F 3 "~" H 3275 5450 50  0001 C CNN
 	1    3275 5450
@@
 F 0 "C4" H 3800 2375 50  0000 L CNN
 F 1 "10n" H 3925 2200 50  0000 L CNN
-F 2 "" H 3963 2125 50  0001 C CNN
+F 2 "Capacitor_SMD:C_0603_1608Metric" H 3963 2125 50  0001 C CNN
 F 3 "~" H 3925 2275 50  0001 C CNN
 	1    3925 2275
@@
 F 0 "Y1" H 3175 4218 50  0000 C CNN
 F 1 "8MHz" H 3175 4127 50  0000 C CNN
-F 2 "" H 3175 3950 50  0001 C CNN
+F 2 "Crystal:Crystal_SMD_5032-2Pin_5.0x3.2mm" H 3175 3950 50  0001 C CNN
 F 3 "~" H 3175 3950 50  0001 C CNN
 	1    3175 3950
@@
 F 0 "C2" H 3310 4104 50  0000 R CNN
 F 1 "33p" H 3310 4195 50  0000 R CNN
-F 2 "" H 3463 4000 50  0001 C CNN
+F 2 "Capacitor_SMD:C_0603_1608Metric" H 3463 4000 50  0001 C CNN
 F 3 "~" H 3425 4150 50  0001 C CNN
 	1    3425 4150
@@
 F 0 "C1" H 2810 4104 50  0000 R CNN
 F 1 "33p" H 2810 4195 50  0000 R CNN
-F 2 "" H 2963 4000 50  0001 C CNN
+F 2 "Capacitor_SMD:C_0603_1608Metric" H 2963 4000 50  0001 C CNN
 F 3 "~" H 2925 4150 50  0001 C CNN
 	1    2925 4150
@@
 F 0 "C10" H 5490 2046 50  0000 L CNN
 F 1 "10n" H 5490 1955 50  0000 L CNN
-F 2 "" H 5413 1850 50  0001 C CNN
+F 2 "Capacitor_SMD:C_0603_1608Metric" H 5413 1850 50  0001 C CNN
 F 3 "~" H 5375 2000 50  0001 C CNN
 	1    5375 2000
@@
 F 0 "C3" H 3715 1096 50  0000 L CNN
 F 1 "4.7u" H 3715 1005 50  0000 L CNN
-F 2 "" H 3638 900 50  0001 C CNN
+F 2 "Capacitor_SMD:C_0603_1608Metric" H 3638 900 50  0001 C CNN
 F 3 "~" H 3600 1050 50  0001 C CNN
 	1    3600 1050
@@
 F 0 "C5" H 4065 1096 50  0000 L CNN
 F 1 "4.7u" H 4065 1005 50  0000 L CNN
-F 2 "" H 3988 900 50  0001 C CNN
+F 2 "Capacitor_SMD:C_0603_1608Metric" H 3988 900 50  0001 C CNN
 F 3 "~" H 3950 1050 50  0001 C CNN
 	1    3950 1050
@@
 F 0 "C6" H 4415 1096 50  0000 L CNN
 F 1 "4.7u" H 4415 1005 50  0000 L CNN
-F 2 "" H 4338 900 50  0001 C CNN
+F 2 "Capacitor_SMD:C_0603_1608Metric" H 4338 900 50  0001 C CNN
 F 3 "~" H 4300 1050 50  0001 C CNN
 	1    4300 1050
@@
 F 0 "C7" H 4765 1096 50  0000 L CNN
 F 1 "4.7u" H 4765 1005 50  0000 L CNN
-F 2 "" H 4688 900 50  0001 C CNN
+F 2 "Capacitor_SMD:C_0603_1608Metric" H 4688 900 50  0001 C CNN
 F 3 "~" H 4650 1050 50  0001 C CNN
 	1    4650 1050
@@
 F 0 "Q1" H 1754 1496 50  0000 L CNN
 F 1 "IRLZ14SPBF" H 1754 1405 50  0000 L CNN
-F 2 "Package_TO_SOT_THT:TO-220-3_Vertical" H 1800 1375 50  0001 L CIN
+F 2 "Package_TO_SOT_SMD:TO-252-2" H 1800 1375 50  0001 L CIN
 F 3 "http://www.infineon.com/dgdl/irlz34npbf.pdf?fileId=5546d462533600a40153567206892720" H 1550 1450 50  0001 L CNN
 	1    1550 1450
@@
 F 0 "Q2" H 1754 2346 50  0000 L CNN
 F 1 "IRLZ14SPBF" H 1754 2255 50  0000 L CNN
-F 2 "Package_TO_SOT_THT:TO-220-3_Vertical" H 1800 2225 50  0001 L CIN
+F 2 "Package_TO_SOT_SMD:TO-252-2" H 1800 2225 50  0001 L CIN
 F 3 "http://www.infineon.com/dgdl/irlz34npbf.pdf?fileId=5546d462533600a40153567206892720" H 1550 2300 50  0001 L CNN
 	1    1550 2300
@@
 F 0 "R5" V 6143 5450 50  0000 C CNN
 F 1 "10K" V 6234 5450 50  0000 C CNN
-F 2 "" V 6280 5450 50  0001 C CNN
+F 2 "Resistor_SMD:R_0603_1608Metric" V 6280 5450 50  0001 C CNN
 F 3 "~" H 6350 5450 50  0001 C CNN
 	1    6350 5450
@@
 F 0 "R4" V 6018 2650 50  0000 C CNN
 F 1 "10K" V 6109 2650 50  0000 C CNN
-F 2 "" V 6155 2650 50  0001 C CNN
+F 2 "Resistor_SMD:R_0603_1608Metric" V 6155 2650 50  0001 C CNN
 F 3 "~" H 6225 2650 50  0001 C CNN
 	1    6225 2650
@@
 F 0 "J2" H 10455 5892 50  0000 L CNN
 F 1 "Conn_01x06" H 10455 5801 50  0000 L CNN
-F 2 "" H 10375 5900 50  0001 C CNN
+F 2 "Connector:Tag-Connect_TC2030-IDC-NL_2x03_P1.27mm_Vertical" H 10375 5900 50  0001 C CNN
 F 3 "~" H 10375 5900 50  0001 C CNN
 	1    10375 5900
@@
 F 0 "J1" H 10375 5567 50  0000 C CNN
 F 1 "Conn_02x05_Odd_Even" H 10375 5476 50  0000 C CNN
-F 2 "" H 10325 5150 50  0001 C CNN
+F 2 "Connector_PinHeader_1.27mm:PinHeader_2x05_P1.27mm_Vertical_SMD" H 10325 5150 50  0001 C CNN
 F 3 "~" H 10325 5150 50  0001 C CNN
 	1    10325 5150
@@
 P 5000 1050
 F 0 "C8" H 5115 1096 50  0000 L CNN
-F 1 "10u" H 5115 1005 50  0000 L CNN
-F 2 "" H 5038 900 50  0001 C CNN
+F 1 "4.7u" H 5115 1005 50  0000 L CNN
+F 2 "Capacitor_SMD:C_0603_1608Metric" H 5038 900 50  0001 C CNN
 F 3 "~" H 5000 1050 50  0001 C CNN
 	1    5000 1050
 	1    0    0    -1
 $EndComp
-$Comp
-L Device:C C9
-U 1 1 6106E847
-P 5350 1050
-F 0 "C9" H 5465 1096 50  0000 L CNN
-F 1 "10u" H 5465 1005 50  0000 L CNN
-F 2 "" H 5388 900 50  0001 C CNN
-F 3 "~" H 5350 1050 50  0001 C CNN
-	1    5350 1050
-	1    0    0    -1
-$EndComp
-$Comp
-L Device:C C11
-U 1 1 6106E851
-P 5700 1050
-F 0 "C11" H 5815 1096 50  0000 L CNN
-F 1 "10u" H 5815 1005 50  0000 L CNN
-F 2 "" H 5738 900 50  0001 C CNN
-F 3 "~" H 5700 1050 50  0001 C CNN
-	1    5700 1050
-	1    0    0    -1
-$EndComp
 Wire Wire Line
 	4650 850  5000 850
 Wire Wire Line
-	5700 850  5700 900
-Wire Wire Line
-	5350 900  5350 850
-Connection ~ 5350 850
-Wire Wire Line
 	5000 850  5000 900
-Connection ~ 5000 850
-Wire Wire Line
-	5000 850  5350 850
 Wire Wire Line
 	4650 1250 5000 1250
 Wire Wire Line
 	5000 1250 5000 1200
-Wire Wire Line
-	5000 1250 5350 1250
-Wire Wire Line
-	5350 1250 5350 1200
-Connection ~ 5000 1250
-Wire Wire Line
-	5700 1250 5700 1200
-Connection ~ 5350 1250
 Connection ~ 4650 850
 Connection ~ 4650 1250
-$Comp
-L Device:C C13
-U 1 1 6108071E
-P 6025 1050
-F 0 "C13" H 6140 1096 50  0000 L CNN
-F 1 "10u" H 6140 1005 50  0000 L CNN
-F 2 "" H 6063 900 50  0001 C CNN
-F 3 "~" H 6025 1050 50  0001 C CNN
-	1    6025 1050
-	1    0    0    -1
-$EndComp
-Wire Wire Line
-	6025 850  6025 900
-Wire Wire Line
-	6025 1250 6025 1200
-Wire Wire Line
-	5350 850  5700 850
-Wire Wire Line
-	5350 1250 5700 1250
 $Comp
 L Device:C C12
@@
 F 0 "C12" H 5915 2046 50  0000 L CNN
 F 1 "4.7u" H 5915 1955 50  0000 L CNN
-F 2 "" H 5838 1850 50  0001 C CNN
+F 2 "Capacitor_SMD:C_0603_1608Metric" H 5838 1850 50  0001 C CNN
 F 3 "~" H 5800 2000 50  0001 C CNN
 	1    5800 2000
@@
 F 0 "FB1" V 6399 1800 50  0000 C CNN
 F 1 "Ferrite_Bead" V 6308 1800 50  0000 C CNN
-F 2 "" V 6055 1800 50  0001 C CNN
+F 2 "Capacitor_SMD:C_0805_2012Metric" V 6055 1800 50  0001 C CNN
 F 3 "~" H 6125 1800 50  0001 C CNN
 	1    6125 1800
@@
 F 0 "R1" H 3195 2596 50  0000 L CNN
 F 1 "10k" H 3195 2505 50  0000 L CNN
-F 2 "" V 3055 2550 50  0001 C CNN
+F 2 "Resistor_SMD:R_0603_1608Metric" V 3055 2550 50  0001 C CNN
 F 3 "~" H 3125 2550 50  0001 C CNN
 	1    3125 2550
@@
 F 0 "SW2" V 3354 2473 50  0000 L CNN
 F 1 "SW_Push" V 3445 2473 50  0000 L CNN
-F 2 "" H 3400 2525 50  0001 C CNN
+F 2 "Button_Switch_SMD:SW_SPST_EVQQ2" H 3400 2525 50  0001 C CNN
 F 3 "~" H 3400 2525 50  0001 C CNN
 	1    3400 2325
@@
 F 0 "R3" H 3720 2996 50  0000 L CNN
 F 1 "10k" H 3720 2905 50  0000 L CNN
-F 2 "" V 3580 2950 50  0001 C CNN
+F 2 "Resistor_SMD:R_0603_1608Metric" V 3580 2950 50  0001 C CNN
 F 3 "~" H 3650 2950 50  0001 C CNN
 	1    3650 2950
@@
 F 0 "SW1" H 3550 2825 50  0000 C CNN
 F 1 "SW_Push" H 3350 2675 50  0000 C CNN
-F 2 "" H 3350 2950 50  0001 C CNN
+F 2 "Button_Switch_SMD:SW_SPST_EVQQ2" H 3350 2950 50  0001 C CNN
 F 3 "~" H 3350 2950 50  0001 C CNN
 	1    3350 2750
@@
 	3550 2750 3650 2750
 Connection ~ 3650 2750
-Connection ~ 5700 1250
-Wire Wire Line
-	5700 1250 6025 1250
-Connection ~ 5700 850
-Wire Wire Line
-	5700 850  6025 850
 Wire Wire Line
 	5575 4250 6025 4250
